Commit message: Adapted xacro
git-svn-id: https://roboticssrv.wtb.tue.nl/svn/ros/user/sjoerd/better_robot_descriptions/amigo_description@17843 3a3c2cfb-d3b9-409e-9e75-db8fcdbcaac6

File: urdf/xacro/amigo_no_wheels.urdf.xacro (robot description, xacro)
@@ -20,5 +20,5 @@
 <include filename="$(find amigo_description)/urdf/xacro/head/head.urdf.xacro" />
 <!--========BUILD KINECT======-->
-<include filename="$(find amigo_description)/urdf/xacro/kinect/kinect.urdf.xacro" />
+<include filename="$(find amigo_description)/urdf/xacro/kinect/top_kinect.urdf.xacro" />
 <include filename="$(find amigo_description)/urdf/xacro/kinect/base_kinect.urdf.xacro" />
 <!--========BUILD ARMS======-->

File: urdf/xacro/arms/arm.urdf.xacro (robot description, xacro)
@@ -41,5 +41,5 @@
    <origin xyz="-0.00959 -0.19131 -0.00001" rpy="0 0 3.1415" />
    <inertia ixx="0.027"  ixy="0"  ixz="0" iyy="0.027" iyz="0" izz="0.004" />
-   <mesh filename="package://amigo_robot_model_groovy/Media/meshes/upperarmtextured.dae" scale="0.0004 0.0004 0.0004"/>
+   <mesh filename="package://amigo_description/media/meshes/upperarmtextured.dae" scale="0.0004 0.0004 0.0004"/>
 </xacro:my_link_texturedmesh>
 <!--the elbow
@@ -56,5 +56,5 @@
    <origin xyz="0.00425 -0.14868 0.00547" rpy="0 -1.5708 0" />
    <inertia ixx="0.0054"  ixy="0"  ixz="0" iyy="0.0054" iyz="0" izz="0.0004" />
-   <mesh filename="package://amigo_robot_model_groovy/Media/meshes/forearmtextured.dae" scale="0.0004 0.0004 0.0004"/>
+   <mesh filename="package://amigo_description/media/meshes/forearmtextured.dae" scale="0.0004 0.0004 0.0004"/>
 </xacro:my_link_texturedmesh>
 <!--the wrist

File: urdf/xacro/body/body.urdf.xacro (robot description, xacro)
@@ -10,5 +10,5 @@
    <origin xyz="0.045 0.0 0.06" rpy="-1.5708 0 -1.5708" />
    <inertia ixx="0.01"  ixy="0"  ixz="0" iyy="0.01" iyz="0" izz="0.01" />
-   <mesh filename="package://amigo_robot_model_groovy/Media/meshes/torsocovers.dae" scale="0.0004 0.0004 0.0004"/>
+   <mesh filename="package://amigo_description/media/meshes/torsocovers.dae" scale="0.0004 0.0004 0.0004"/>
 </xacro:my_link_texturedmesh>
 <!--the spindle-->
@@ -17,5 +17,5 @@
    <origin xyz="0.05 0 0.0" rpy="0 0 1.5708"/>
    <inertia ixx="0.01"  ixy="0"  ixz="0" iyy="0.01" iyz="0" izz="0.01" />
-   <mesh filename="package://amigo_robot_model_groovy/Media/meshes/torsoslidertextured.dae" scale="0.004 0.004 0.004"/>
+   <mesh filename="package://amigo_description/media/meshes/torsoslidertextured.dae" scale="0.004 0.004 0.004"/>
 </xacro:my_link_texturedmesh>
 <!--the bottomcover -->
@@ -24,5 +24,5 @@
    <origin xyz="0.0 0.0 0.23" rpy="0 0 -1.5708" />
    <inertia ixx="2.63"  ixy="0"  ixz="0" iyy="2.63" iyz="0" izz="2.4" />
-   <mesh filename="package://amigo_robot_model_groovy/Media/meshes/bottomcovers.dae" scale="0.0004 0.0004 0.0004"/>
+   <mesh filename="package://amigo_description/media/meshes/bottomcovers.dae" scale="0.0004 0.0004 0.0004"/>
 </xacro:my_link_texturedmesh>
 <!--the root of the tf-tree, because it serves only this function it has no visuals-->

File: urdf/xacro/body_extra_visuals/body_extra.urdf.xacro (robot description, xacro)
@@ -23,5 +23,5 @@
    <origin xyz="-0.4  0.0 0.0" rpy="0 1.5708 0"/>
    <inertia ixx="0.01"  ixy="0"  ixz="0" iyy="0.01" iyz="0" izz="0.01" />
-   <mesh filename="package://amigo_robot_model_groovy/Media/meshes/torsoassistslidertextured.dae" scale="0.004 0.004 0.005"/>
+   <mesh filename="package://amigo_description/media/meshes/torsoassistslidertextured.dae" scale="0.004 0.004 0.005"/>
 </xacro:my_link_texturedmesh>
 <!--left link-->
@@ -30,5 +30,5 @@
    <origin xyz="-0.4  0.0 0.0" rpy="0 1.5708 0"/>
    <inertia ixx="0.01"  ixy="0"  ixz="0" iyy="0.01" iyz="0" izz="0.01" />
-   <mesh filename="package://amigo_robot_model_groovy/Media/meshes/torsoassistslidertextured.dae" scale="0.004 0.004 0.005"/>
+   <mesh filename="package://amigo_description/media/meshes/torsoassistslidertextured.dae" scale="0.004 0.004 0.005"/>
 </xacro:my_link_texturedmesh>
 <!--back link-->
@@ -37,5 +37,5 @@
    <origin xyz="-0.4 0.0 0.0" rpy="0 1.5708 0"/>
    <inertia ixx="0.01"  ixy="0"  ixz="0" iyy="0.01" iyz="0" izz="0.01" />
-   <mesh filename="package://amigo_robot_model_groovy/Media/meshes/torsoassistslidertextured.dae" scale="0.004 0.004 0.005"/>
+   <mesh filename="package://amigo_description/media/meshes/torsoassistslidertextured.dae" scale="0.004 0.004 0.005"/>
 </xacro:my_link_texturedmesh>
 <!--left joint-->

File: urdf/xacro/head/head.urdf.xacro (robot description, xacro)
@@ -32,5 +32,5 @@
    <origin xyz="0.0 -0.0 0.015" rpy="0 0 0" />
    <inertia ixx="0.001"  ixy="0"  ixz="0" iyy="0.001" iyz="0" izz="0.001" />
-   <mesh filename="package://amigo_robot_model_groovy/Media/meshes/necktilttextured.dae" scale="0.004 0.004 0.004"/>
+   <mesh filename="package://amigo_description/media/meshes/necktilttextured.dae" scale="0.004 0.004 0.004"/>
 </xacro:my_link_texturedmesh>
 <!--the head itself-->
@@ -39,5 +39,5 @@
    <origin xyz="0.0 0.0 0.141" rpy="0 0 -1.5708"/>
    <inertia ixx="0"  ixy="0"  ixz="0" iyy="0" iyz="0" izz="0" />
-   <mesh filename="package://amigo_robot_model_groovy/Media/meshes/headtextured.dae" scale="0.0004 0.0004 0.0004"/>
+   <mesh filename="package://amigo_description/media/meshes/headtextured.dae" scale="0.0004 0.0004 0.0004"/>
   </my_link_texturedmesh>
   <joint name="head_joint" type="fixed">

File: urdf/xacro/kinect/base_kinect.urdf.xacro (robot description, xacro)
@@ -5,10 +5,10 @@
       xmlns:xacro="http://ros.org/wiki/xacro">
   <property name="M_PI" value="3.14159"/>
-  <joint name="base_kinect_base_kinect_joint" type="fixed">
+  <joint name="base_kinect/base_kinect_joint" type="fixed">
     <origin xyz="0.3 0 0.26" rpy="0 -0.07 0" /> <!-- THESE VALUES STILL HAVE TO BE CALIBRATED!! -->
     <parent link="base" />
-    <child link="base_kinect_openni_camera" />
+    <child link="base_kinect/openni_camera" />
   </joint>
-  <link name="base_kinect_openni_camera">
+  <link name="base_kinect/openni_camera">
     <inertial>
       <mass value="0.01" />
@@ -23,5 +23,5 @@
 	<!--<box size="0 0 0"/>-->
         <!--mesh filename="package://amigo_robot_model_groovy/description/kinect/meshes/kinect.dae" scale="0.001 0.001 0.001"/-->
-        <mesh filename="package://amigo_robot_model_groovy/description/kinect/meshes/kinect_without_base.dae"/>
+        <mesh filename="package://amigo_description/media/meshes/kinect/kinect_without_base.dae"/>
       </geometry>
     </visual>
@@ -31,14 +31,14 @@
 	<!--<box size="0.01 0.01 0.01"/>-->
         <!--<mesh filename="package://amigo_robot_model_groovy/description/kinect/meshes/kinect.dae" scale="0.001 0.001 0.001"/>-->
-        <mesh filename="package://amigo_robot_model_groovy/description/kinect/meshes/kinect_without_base.dae"/>
+        <mesh filename="package://amigo_description/media/meshes/kinect/kinect_without_base.dae"/>
       </geometry>
     </collision>
   </link>
-  <joint name="base_kinect_kinect_depth_joint" type="fixed">
+  <joint name="base_kinect/kinect_depth_joint" type="fixed">
     <origin xyz="0 0.018 0" rpy="0 0 0" />
-    <parent link="base_kinect_openni_camera" />
-    <child link="base_kinect_openni_depth_frame" />
+    <parent link="base_kinect/openni_camera" />
+    <child link="base_kinect/openni_depth_frame" />
   </joint>
-  <link name="base_kinect_openni_depth_frame">
+  <link name="base_kinect/openni_depth_frame">
     <inertial>
       <mass value="0.01" />
@@ -49,10 +49,10 @@
     </inertial>
   </link>
-  <joint name="base_kinect_kinect_depth_optical_joint" type="fixed">
+  <joint name="base_kinect/kinect_depth_optical_joint" type="fixed">
     <origin xyz="0 0 0" rpy="${-M_PI/2} 0 ${-M_PI/2}" />
-    <parent link="base_kinect_openni_depth_frame" />
-    <child link="base_kinect_openni_depth_optical_frame" />
+    <parent link="base_kinect/openni_depth_frame" />
+    <child link="base_kinect/openni_depth_optical_frame" />
   </joint>
-  <link name="base_kinect_openni_depth_optical_frame">
+  <link name="base_kinect/openni_depth_optical_frame">
     <inertial>
       <mass value="0.001" />
@@ -63,10 +63,10 @@
     </inertial>
   </link>
-  <joint name="base_kinect_kinect_rgb_joint" type="fixed">
+  <joint name="base_kinect/kinect_rgb_joint" type="fixed">
     <origin xyz="0 -0.005 0" rpy="0 0 0" />
-    <parent link="base_kinect_openni_camera" />
-    <child link="base_kinect_openni_rgb_frame" />
+    <parent link="base_kinect/openni_camera" />
+    <child link="base_kinect/openni_rgb_frame" />
   </joint>
-  <link name="base_kinect_openni_rgb_frame">
+  <link name="base_kinect/openni_rgb_frame">
     <inertial>
       <mass value="0.001" />
@@ -77,10 +77,10 @@
     </inertial>
   </link>
-  <joint name="base_kinect_kinect_rgb_optical_joint" type="fixed">
+  <joint name="base_kinect/kinect_rgb_optical_joint" type="fixed">
     <origin xyz="0 0 0" rpy="${-M_PI/2} 0 ${-M_PI/2}" />
-    <parent link="base_kinect_openni_rgb_frame" />
-    <child link="base_kinect_openni_rgb_optical_frame" />
+    <parent link="base_kinect/openni_rgb_frame" />
+    <child link="base_kinect/openni_rgb_optical_frame" />
   </joint>
-  <link name="base_kinect_openni_rgb_optical_frame">
+  <link name="base_kinect/openni_rgb_optical_frame">
     <inertial>
       <mass value="0.001" />

File: urdf/xacro/kinect/top_kinect.urdf.xacro (robot description, xacro)
@@ -5,10 +5,10 @@
       xmlns:xacro="http://ros.org/wiki/xacro">
   <property name="M_PI" value="3.14159"/>
-  <joint name="base_kinect_joint" type="fixed">
+  <joint name="top_kinect/base_kinect_joint" type="fixed">
     <origin xyz="0.07 0 0.07" rpy="0 0 0" /> <!-- THESE VALUES ARE ROUGH ESTIMATES!! -->
     <parent link="head" />
-    <child link="openni_camera" />
+    <child link="top_kinect/openni_camera" />
   </joint>
-  <link name="openni_camera">
+  <link name="top_kinect/openni_camera">
     <inertial>
       <mass value="0.01" />
@@ -33,10 +33,10 @@
     </collision>-->
   </link>
-  <joint name="kinect_depth_joint" type="fixed">
+  <joint name="top_kinect/kinect_depth_joint" type="fixed">
     <origin xyz="0 0.018 0" rpy="0 0 0" />
-    <parent link="openni_camera" />
-    <child link="openni_depth_frame" />
+    <parent link="top_kinect/openni_camera" />
+    <child link="top_kinect/openni_depth_frame" />
   </joint>
-  <link name="openni_depth_frame">
+  <link name="top_kinect/openni_depth_frame">
     <inertial>
       <mass value="0.01" />
@@ -47,10 +47,10 @@
     </inertial>
   </link>
-  <joint name="kinect_depth_optical_joint" type="fixed">
+  <joint name="top_kinect/kinect_depth_optical_joint" type="fixed">
     <origin xyz="0 0 0" rpy="${-M_PI/2} 0 ${-M_PI/2}" />
-    <parent link="openni_depth_frame" />
-    <child link="openni_depth_optical_frame" />
+    <parent link="top_kinect/openni_depth_frame" />
+    <child link="top_kinect/openni_depth_optical_frame" />
   </joint>
-  <link name="openni_depth_optical_frame">
+  <link name="top_kinect/openni_depth_optical_frame">
     <inertial>
       <mass value="0.001" />
@@ -61,10 +61,10 @@
     </inertial>
   </link>
-  <joint name="kinect_rgb_joint" type="fixed">
+  <joint name="top_kinect/kinect_rgb_joint" type="fixed">
     <origin xyz="0 -0.005 0" rpy="0 0 0" />
-    <parent link="openni_camera" />
-    <child link="openni_rgb_frame" />
+    <parent link="top_kinect/openni_camera" />
+    <child link="top_kinect/openni_rgb_frame" />
   </joint>
-  <link name="openni_rgb_frame">
+  <link name="top_kinect/openni_rgb_frame">
     <inertial>
       <mass value="0.001" />
@@ -75,10 +75,10 @@
     </inertial>
   </link>
-  <joint name="kinect_rgb_optical_joint" type="fixed">
+  <joint name="top_kinect/kinect_rgb_optical_joint" type="fixed">
     <origin xyz="0 0 0" rpy="${-M_PI/2} 0 ${-M_PI/2}" />
-    <parent link="openni_rgb_frame" />
-    <child link="openni_rgb_optical_frame" />
+    <parent link="top_kinect/openni_rgb_frame" />
+    <child link="top_kinect/openni_rgb_optical_frame" />
   </joint>
-  <link name="openni_rgb_optical_frame">
+  <link name="top_kinect/openni_rgb_optical_frame">
     <inertial>
       <mass value="0.001" />

File: urdf/xacro/laser/laser.urdf.xacro (robot description, xacro)
@@ -33,5 +33,5 @@
    <origin xyz="0.025 0.0 -0.14" rpy="0 0 3.1415" />
    <inertia ixx="0.0001"  ixy="0"  ixz="0" iyy="0.0001" iyz="0" izz="0.0001" />
-   <mesh filename="package://amigo_robot_model_groovy/Media/meshes/logo.dae" scale="0.0016 0.0016 0.0016"/>
+   <mesh filename="package://amigo_description/media/meshes/logo.dae" scale="0.0016 0.0016 0.0016"/>
 </xacro:my_link_texturedmesh>
   <joint name="logo_joint" type="fixed">

File: urdf/xacro/materials.urdf.xacro (robot description, xacro)
@@ -30,17 +30,17 @@
   </material>
   <material name="bottomcovers">
-    <texture filename="package://amigo_robot_model_groovy/Media/materials/textures/bottomcovers/finalreduced.jpg" />
+    <texture filename="package://amigo_description/media/materials/textures/bottomcovers/finalreduced.jpg" />
   </material>
     <material name="white">
-    <texture filename="package://amigo_robot_model_groovy/Media/materials/textures/white/white.jpg" />
+    <texture filename="package://amigo_description/media/materials/textures/white/white.jpg" />
   </material>
   <material name="logo">
-    <texture filename="package://amigo_robot_model_groovy/Media/materials/textures/logo/tue.jpg" />
+    <texture filename="package://amigo_description/media/materials/textures/logo/tue.jpg" />
   </material>
   <material name="aluminum">
-    <texture filename="package://amigo_robot_model_groovy/Media/materials/textures/aluminum/aluminium_0001_c.jpg" />
+    <texture filename="package://amigo_description/media/materials/textures/aluminum/aluminium_0001_c.jpg" />
   </material>
   <material name="orange">
-    <texture filename="package://amigo_robot_model_groovy/Media/materials/textures/orange/orange.jpg" />
+    <texture filename="package://amigo_description/media/materials/textures/orange/orange.jpg" />
   </material>
 </robot>
