Commit message: Renamed textures for better sdf conversion
git-svn-id: https://roboticssrv.wtb.tue.nl/svn/ros/code/tue-ros-pkg/trunk/amigo_common/amigo_description@18208 3a3c2cfb-d3b9-409e-9e75-db8fcdbcaac6

File: urdf/xacro/definitions.xacro (robot description, xacro)
@@ -57,5 +57,5 @@
   </link>
 <gazebo reference="${name}">
-      <material>amigo_robot_model_groovy/${texture}</material>
+      <material>amigo_description/${texture}</material>
       <turnGravityOff>false</turnGravityOff>
     </gazebo>
@@ -134,5 +134,5 @@
   </link>
 <gazebo reference="${name}">
-	  <material>amigo_robot_model_groovy/${texture}</material>
+	  <material>amigo_description/${texture}</material>
       <turnGravityOff>false</turnGravityOff>
     </gazebo>
@@ -161,5 +161,5 @@
   </link>
 <gazebo reference="${name}">
-	  <material>amigo_robot_model_groovy/${texture}</material>
+	  <material>amigo_description/${texture}</material>
       <turnGravityOff>false</turnGravityOff>
     </gazebo>

File: urdf/xacro/kinect/base_kinect.urdf.xacro (robot description, xacro)
@@ -22,5 +22,5 @@
       <geometry>
 	<!--<box size="0 0 0"/>-->
-        <!--mesh filename="package://amigo_robot_model_groovy/description/kinect/meshes/kinect.dae" scale="0.001 0.001 0.001"/-->
+        <!--mesh filename="package://amigo_description/description/kinect/meshes/kinect.dae" scale="0.001 0.001 0.001"/-->
         <mesh filename="package://amigo_description/media/meshes/kinect/kinect_without_base.dae"/>
       </geometry>
@@ -30,5 +30,5 @@
       <geometry>
 	<!--<box size="0.01 0.01 0.01"/>-->
-        <!--<mesh filename="package://amigo_robot_model_groovy/description/kinect/meshes/kinect.dae" scale="0.001 0.001 0.001"/>-->
+        <!--<mesh filename="package://amigo_description/description/kinect/meshes/kinect.dae" scale="0.001 0.001 0.001"/>-->
         <mesh filename="package://amigo_description/media/meshes/kinect/kinect_without_base.dae"/>
       </geometry>

File: urdf/xacro/kinect/top_kinect.urdf.xacro (robot description, xacro)
@@ -22,6 +22,6 @@
       <geometry>
 		<box size="0 0 0"/>
-        <!--mesh filename="package://amigo_robot_model_groovy/kinect/meshes/kinect.dae" scale="0.001 0.001 0.001"/-->
-        <!--<mesh filename="package://amigo_robot_model_groovy/kinect/meshes/kinect_without_base.dae"/>-->
+        <!--mesh filename="package://amigo_description/kinect/meshes/kinect.dae" scale="0.001 0.001 0.001"/-->
+        <!--<mesh filename="package://amigo_description/kinect/meshes/kinect_without_base.dae"/>-->
       </geometry>
     </visual>
