Commit message: Added gazebo plugins to xacro
git-svn-id: https://roboticssrv.wtb.tue.nl/svn/ros/code/tue-ros-pkg/trunk/amigo_common/amigo_description@18209 3a3c2cfb-d3b9-409e-9e75-db8fcdbcaac6

File: urdf/xacro/amigo.urdf.xacro (robot description, xacro)
@@ -30,3 +30,5 @@
 <xacro:arm_extra whichside="right" sidesign="+1.0" rollsign="+"/>
 <xacro:arm_extra whichside="left"  sidesign="-1.0" rollsign="-"/>
+<!-- GAZEBO -->
+<include filename="$(find amigo_description)/urdf/xacro/gazebo.urdf.xacro"/>
 </robot>

File: urdf/xacro/arms/arm.urdf.xacro (robot description, xacro)
@@ -37,5 +37,5 @@
 </xacro:my_link>
 <!--the upper arm-->
-<xacro:my_link_texturedmesh name="upper_arm_${whichside}" mass="2.95" texture="white">
+<xacro:my_link_texturedmesh name="upper_arm_${whichside}" mass="2.95" texture="amigo_description/white">
    <origin xyz="0.0 -0.2 0.0" rpy="0 0 0"/>
    <origin xyz="-0.00959 -0.19131 -0.00001" rpy="0 0 3.1415" />
@@ -52,5 +52,5 @@
 </xacro:my_link>
 <!--the forearm-->
-<xacro:my_link_texturedmesh name="fore_arm_${whichside}" mass="0.85" texture="white">
+<xacro:my_link_texturedmesh name="fore_arm_${whichside}" mass="0.85" texture="amigo_description/white">
    <origin xyz="0.0 -0.14 0.0" rpy="0.0 0 0"/>
    <origin xyz="0.00425 -0.14868 0.00547" rpy="0 -1.5708 0" />

File: urdf/xacro/body/body.urdf.xacro (robot description, xacro)
@@ -6,5 +6,5 @@
 <!--links start here-->
 <!--the torso-->
-<xacro:my_link_texturedmesh name="torso" mass="16" texture="white">
+<xacro:my_link_texturedmesh name="torso" mass="16" texture="amigo_description/white">
    <origin xyz="0.0 0.0 0.0" rpy="0 0 0"/>
    <origin xyz="0.045 0.0 0.06" rpy="-1.5708 0 -1.5708" />
@@ -20,5 +20,5 @@
 </xacro:my_link_texturedmesh>
 <!--the bottomcover -->
-<xacro:my_link_texturedmesh name="base" mass="20" texture="bottomcovers">
+<xacro:my_link_texturedmesh name="base" mass="20" texture="amigo_description/bottomcovers">
    <origin xyz="0.0 0.0 0.3275" rpy="0 0 0"/>
    <origin xyz="0.0 0.0 0.23" rpy="0 0 -1.5708" />

File: urdf/xacro/definitions.xacro (robot description, xacro)
@@ -57,5 +57,5 @@
   </link>
 <gazebo reference="${name}">
-      <material>amigo_description/${texture}</material>
+      <material>${texture}</material>
       <turnGravityOff>false</turnGravityOff>
     </gazebo>
@@ -134,5 +134,5 @@
   </link>
 <gazebo reference="${name}">
-	  <material>amigo_description/${texture}</material>
+	  <material>${texture}</material>
       <turnGravityOff>false</turnGravityOff>
     </gazebo>
@@ -161,5 +161,5 @@
   </link>
 <gazebo reference="${name}">
-	  <material>amigo_description/${texture}</material>
+	  <material>${texture}</material>
       <turnGravityOff>false</turnGravityOff>
     </gazebo>

File: urdf/xacro/laser/laser.urdf.xacro (robot description, xacro)
@@ -29,5 +29,5 @@
 </joint>
 <!--the tue logo in front of the laser-->
-<xacro:my_link_texturedmesh name="logo" mass="0.01" texture="logo">
+<xacro:my_link_texturedmesh name="logo" mass="0.01" texture="amigo_description/logo">
    <origin xyz="0.0 0.0 0.0" rpy="0 0 0"/>
    <origin xyz="0.025 0.0 -0.14" rpy="0 0 3.1415" />

File: urdf/xacro/materials.urdf.xacro (robot description, xacro)
@@ -29,17 +29,17 @@
     <color rgba="0.6 0.6 0.6 1.0"/>
   </material>
-  <material name="bottomcovers">
+  <material name="amigo_description/bottomcovers">
     <texture filename="package://amigo_description/media/materials/textures/bottomcovers/finalreduced.jpg" />
   </material>
-    <material name="white">
+    <material name="amigo_description/white">
     <texture filename="package://amigo_description/media/materials/textures/white/white.jpg" />
   </material>
-  <material name="logo">
+  <material name="amigo_description/logo">
     <texture filename="package://amigo_description/media/materials/textures/logo/tue.jpg" />
   </material>
-  <material name="aluminum">
+  <material name="amigo_description/aluminum">
     <texture filename="package://amigo_description/media/materials/textures/aluminum/aluminium_0001_c.jpg" />
   </material>
-  <material name="orange">
+  <material name="amigo_description/orange">
     <texture filename="package://amigo_description/media/materials/textures/orange/orange.jpg" />
   </material>
