Commit message: added Orange to the material list

File: urdf/xacro/materials.urdf.xacro (robot description, xacro)
@@ -29,4 +29,7 @@
     <color rgba="0.6 0.6 0.6 1.0"/>
   </material>
+  <material name="Orange">
+    <color rgba="1.0 0.33 0.0"/>
+  </material>
   <material name="amigo_description/bottomcovers">
     <texture filename="package://amigo_description/media/materials/textures/bottomcovers/finalreduced.jpg" />
