Commit message: Updated amigo urdf; can now spawn amigo using launch file
git-svn-id: https://roboticssrv.wtb.tue.nl/svn/ros/user/sjoerd/better_robot_descriptions/amigo_description@17832 3a3c2cfb-d3b9-409e-9e75-db8fcdbcaac6

File: urdf/amigo_no_wheels.urdf (robot description, URDF)
Before this commit: robot amigo, 78 links, 77 joints
Links:
- link base: geometry collision mesh filename=package://amigo_description/media/meshes/bottomcovers.dae scale=0.0004 0.0004 0.0004; visual mesh filename=package://amigo_description/media/meshes/bottomcovers.dae scale=0.0004 0.0004 0.0004
- link base_kinect_openni_camera: geometry collision mesh filename=package://amigo_description/media/meshes/kinect/kinect_with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; visual mesh filename=package://amigo_description/media/meshes/kinect/kinect_with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
- link fore_arm_left: geometry collision mesh filename=package://amigo_description/media/meshes/forearmtextured.dae scale=0.0004 0.0004 0.0004; visual mesh filename=package://amigo_description/media/meshes/forearmtextured.dae scale=0.0004 0.0004 0.0004
- link fore_arm_right: geometry collision mesh filename=package://amigo_description/media/meshes/forearmtextured.dae scale=0.0004 0.0004 0.0004; visual mesh filename=package://amigo_description/media/meshes/forearmtextured.dae scale=0.0004 0.0004 0.0004
- link head: geometry collision mesh filename=package://amigo_description/media/meshes/headtextured.dae scale=0.0004 0.0004 0.0004; visual mesh filename=package://amigo_description/media/meshes/headtextured.dae scale=0.0004 0.0004 0.0004
- link logo: geometry collision mesh filename=package://amigo_description/media/meshes/logo.dae scale=0.0016 0.0016 0.0016; visual mesh filename=package://amigo_description/media/meshes/logo.dae scale=0.0016 0.0016 0.0016
- link neck_tilt: geometry collision mesh filename=package://amigo_description/media/meshes/necktilttextured.d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 scale=0.004 0.004 0.004; visual mesh filename=package://amigo_description/media/meshes/necktilttextured.d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 scale=0.004 0.004 0.004
- link torso: geometry collision mesh filename=package://amigo_description/media/meshes/torsocovers.dae scale=0.0004 0.0004 0.0004; visual mesh filename=package://amigo_description/media/meshes/torsocovers.dae scale=0.0004 0.0004 0.0004
- link torso_assist_slider_back: geometry collision mesh filename=package://amigo_description/media/meshes/torsoassistslidert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 scale=0.004 0.004 0.005; visual mesh filename=package://amigo_description/media/meshes/torsoassistslidert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 scale=0.004 0.004 0.005
- link torso_assist_slider_left: geometry collision mesh filename=package://amigo_description/media/meshes/torsoassistslidert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 scale=0.004 0.004 0.005; visual mesh filename=package://amigo_description/media/meshes/torsoassistslidert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 scale=0.004 0.004 0.005
- link torso_assist_slider_right: geometry collision mesh filename=package://amigo_description/media/meshes/torsoassistslidert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 scale=0.004 0.004 0.005; visual mesh filename=package://amigo_description/media/meshes/torsoassistslidert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 scale=0.004 0.004 0.005
- link torso_slider: geometry collision mesh filename=package://amigo_description/media/meshes/torsoslidertexture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 scale=0.004 0.004 0.004; visual mesh filename=package://amigo_description/media/meshes/torsoslidertexture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 scale=0.004 0.004 0.004
- link upper_arm_left: geometry collision mesh filename=package://amigo_description/media/meshes/upperarmtextured.d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 scale=0.0004 0.0004 0.0004; visual mesh filename=package://amigo_description/media/meshes/upperarmtextured.d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 scale=0.0004 0.0004 0.0004
- link upper_arm_right: geometry collision mesh filename=package://amigo_description/media/meshes/upperarmtextured.d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 scale=0.0004 0.0004 0.0004; visual mesh filename=package://amigo_description/media/meshes/upperarmtextured.d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 scale=0.0004 0.0004 0.0004

Commit message: Fixed kinect link names (for better tf tree)
git-svn-id: https://roboticssrv.wtb.tue.nl/svn/ros/user/sjoerd/better_robot_descriptions/amigo_description@17835 3a3c2cfb-d3b9-409e-9e75-db8fcdbcaac6

File: urdf/amigo_no_wheels.urdf (robot description, URDF)
Before this commit: robot amigo, 78 links, 77 joints
Links:
- removed link base_kinect_openni_camera
- removed link base_kinect_openni_depth_frame
- removed link base_kinect_openni_depth_optical_frame
- removed link base_kinect_openni_rgb_frame
- removed link base_kinect_openni_rgb_optical_frame
- removed link openni_camera
- removed link openni_depth_frame
- removed link openni_depth_optical_frame
- removed link openni_rgb_frame
- removed link openni_rgb_optical_frame
- added link base_kinect/openni_camera, mass 0.01; collision mesh filename=package://amigo_description/media/meshes/kinect/kinect_with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; visual mesh filename=package://amigo_description/media/meshes/kinect/kinect_with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
- added link base_kinect/openni_depth_frame, mass 0.01
- added link base_kinect/openni_depth_optical_frame, mass 0.001
- added link base_kinect/openni_rgb_frame, mass 0.001
- added link base_kinect/openni_rgb_optical_frame, mass 0.001
- added link top_kinect/openni_camera, mass 0.01; visual box size=0 0 0
- added link top_kinect/openni_depth_frame, mass 0.01
- added link top_kinect/openni_depth_optical_frame, mass 0.001
- added link top_kinect/openni_rgb_frame, mass 0.001
- added link top_kinect/openni_rgb_optical_frame, mass 0.001
Joints:
- removed joint base_kinect_kinect_depth_optical_joint
- removed joint base_kinect_kinect_rgb_joint
- removed joint base_kinect_kinect_rgb_optical_joint
- removed joint kinect_depth_joint
- removed joint kinect_depth_optical_joint
- removed joint kinect_rgb_joint
- removed joint kinect_rgb_optical_joint
- added joint base_kinect/kinect_depth_optical_joint: type fixed, parent base_kinect/openni_depth_frame, child base_kinect/openni_depth_optical_frame, origin xyz=0 0 0 rpy=-1.570795 0 -1.570795
- added joint base_kinect/kinect_rgb_joint: type fixed, parent base_kinect/openni_camera, child base_kinect/openni_rgb_frame, origin xyz=0 -0.005 0 rpy=0 0 0
- added joint base_kinect/kinect_rgb_optical_joint: type fixed, parent base_kinect/openni_rgb_frame, child base_kinect/openni_rgb_optical_frame, origin xyz=0 0 0 rpy=-1.570795 0 -1.570795
- added joint top_kinect/kinect_depth_joint: type fixed, parent top_kinect/openni_camera, child top_kinect/openni_depth_frame, origin xyz=0 0.018 0 rpy=0 0 0
- added joint top_kinect/kinect_depth_optical_joint: type fixed, parent top_kinect/openni_depth_frame, child top_kinect/openni_depth_optical_frame, origin xyz=0 0 0 rpy=-1.570795 0 -1.570795
- added joint top_kinect/kinect_rgb_joint: type fixed, parent top_kinect/openni_camera, child top_kinect/openni_rgb_frame, origin xyz=0 -0.005 0 rpy=0 0 0
- added joint top_kinect/kinect_rgb_optical_joint: type fixed, parent top_kinect/openni_rgb_frame, child top_kinect/openni_rgb_optical_frame, origin xyz=0 0 0 rpy=-1.570795 0 -1.570795
- joint base_kinect_base_kinect_joint: child base_kinect_openni_camera -> base_kinect/openni_camera
- joint base_kinect_joint: child openni_camera -> top_kinect/openni_camera
- joint base_kinect_kinect_depth_joint: child base_kinect_openni_depth_frame -> base_kinect/openni_depth_frame; parent base_kinect_openni_camera -> base_kinect/openni_camera

Commit message: Now uses xacrod file
git-svn-id: https://roboticssrv.wtb.tue.nl/svn/ros/user/sjoerd/better_robot_descriptions/amigo_description@17849 3a3c2cfb-d3b9-409e-9e75-db8fcdbcaac6

File: urdf/amigo_no_wheels.urdf (robot description, URDF)
Before this commit: robot amigo, 78 links, 77 joints
Links:
- removed link base_fixed_link
- removed link base_x_link
- removed link base_y_link
- removed link hand_marker_left
- removed link hand_marker_right
- removed link world
Joints:
- removed joint base_fixed_joint
- removed joint base_kinect_base_kinect_joint
- removed joint base_kinect_joint
- removed joint base_kinect_kinect_depth_joint
- removed joint base_phi_joint
- removed joint base_x_joint
- removed joint base_y_joint
- removed joint marker_joint_left
- removed joint marker_joint_right
- added joint base_kinect/base_kinect_joint: type fixed, parent base, child base_kinect/openni_camera, origin xyz=0.3 0 0.26 rpy=0 -0.07 0
- added joint base_kinect/kinect_depth_joint: type fixed, parent base_kinect/openni_camera, child base_kinect/openni_depth_frame, origin xyz=0 0.018 0 rpy=0 0 0
- added joint top_kinect/base_kinect_joint: type fixed, parent head, child top_kinect/openni_camera, origin xyz=0.07 0 0.07 rpy=0 0 0
