Commit message: Renamed some files
git-svn-id: https://roboticssrv.wtb.tue.nl/svn/ros/code/tue-ros-pkg/trunk/amigo_common/amigo_description@18200 3a3c2cfb-d3b9-409e-9e75-db8fcdbcaac6

File: urdf/amigo.urdf (robot description, URDF)
Before this commit: robot amigo, 72 links, 71 joints
Links:
- link finger1_left: mass 0.05 -> 0.01
- link finger1_right: mass 0.05 -> 0.01
- link finger1_tip_left: mass 0.05 -> 0.01
- link finger1_tip_right: mass 0.05 -> 0.01
- link finger2_left: mass 0.05 -> 0.01
- link finger2_right: mass 0.05 -> 0.01
- link finger2_tip_left: mass 0.05 -> 0.01
- link finger2_tip_right: mass 0.05 -> 0.01
- link fore_arm_left: mass 0.1 -> 0.85
- link fore_arm_right: mass 0.1 -> 0.85
- link shoulder_link1_left: mass 0.1 -> 0.25
- link shoulder_link1_right: mass 0.1 -> 0.25
- link shoulder_link2_left: mass 0.1 -> 0.15
- link shoulder_link2_right: mass 0.1 -> 0.15
- link shoulder_mount_left: mass 0.1 -> 0.15
- link shoulder_mount_right: mass 0.1 -> 0.15
- link upper_arm_left: mass 2.9 -> 2.95
- link upper_arm_right: mass 2.9 -> 2.95

Commit message: Renamed some files
git-svn-id: https://roboticssrv.wtb.tue.nl/svn/ros/code/tue-ros-pkg/trunk/amigo_common/amigo_description@18201 3a3c2cfb-d3b9-409e-9e75-db8fcdbcaac6

File: urdf/amigo.urdf (robot description, URDF)
Before this commit: robot amigo, 72 links, 71 joints
Links:
- link finger1_left: mass 0.01 -> 0.05
- link finger1_right: mass 0.01 -> 0.05
- link finger1_tip_left: mass 0.01 -> 0.05
- link finger1_tip_right: mass 0.01 -> 0.05
- link finger2_left: mass 0.01 -> 0.05
- link finger2_right: mass 0.01 -> 0.05
- link finger2_tip_left: mass 0.01 -> 0.05
- link finger2_tip_right: mass 0.01 -> 0.05
- link fore_arm_left: mass 0.85 -> 0.1
- link fore_arm_right: mass 0.85 -> 0.1
- link shoulder_link1_left: mass 0.25 -> 0.1
- link shoulder_link1_right: mass 0.25 -> 0.1
- link shoulder_link2_left: mass 0.15 -> 0.1
- link shoulder_link2_right: mass 0.15 -> 0.1
- link shoulder_mount_left: mass 0.15 -> 0.1
- link shoulder_mount_right: mass 0.15 -> 0.1
- link upper_arm_left: mass 2.95 -> 2.9
- link upper_arm_right: mass 2.95 -> 2.9

Commit message: Updated generated sdf and urdf
git-svn-id: https://roboticssrv.wtb.tue.nl/svn/ros/code/tue-ros-pkg/trunk/amigo_common/amigo_description@18253 3a3c2cfb-d3b9-409e-9e75-db8fcdbcaac6

File: urdf/amigo.urdf (robot description, URDF)
Before this commit: robot amigo, 72 links, 71 joints
Joints:
- joint spindle_joint: limit lower=0.0 upper=0.41 effort=30 velocity=1.0 -> lower=0.0 upper=0.41 effort=1000 velocity=10.0

Commit message: Updated models
git-svn-id: https://roboticssrv.wtb.tue.nl/svn/ros/code/tue-ros-pkg/trunk/amigo_common/amigo_description@18353 3a3c2cfb-d3b9-409e-9e75-db8fcdbcaac6

File: urdf/amigo.urdf (robot description, URDF)
Before this commit: robot amigo, 72 links, 71 joints
Joints:
- removed joint spindle_joint
- added joint torso_joint: type prismatic, parent base, child torso_slider, origin xyz=0.0 0.0 0.58 rpy=3.14159265 -1.5708 0, axis 1 0 0, limit lower=0.0 upper=0.41 effort=1000 velocity=10.0

File: urdf/xacro/body/body.urdf.xacro (robot description, xacro)
@@ -34,5 +34,5 @@
 </xacro:my_link>
 <!-- joints start here -->
-<joint name="spindle_joint" type="prismatic">
+<joint name="torso_joint" type="prismatic">
   <parent link="base"/>
   <child link="torso_slider"/>

Commit message: Added torso laser
git-svn-id: https://roboticssrv.wtb.tue.nl/svn/ros/code/tue-ros-pkg/trunk/amigo_common/amigo_description@18394 3a3c2cfb-d3b9-409e-9e75-db8fcdbcaac6

File: urdf/amigo.urdf (robot description, URDF)
Before this commit: robot amigo, 72 links, 71 joints
Links:
- added link torso_dummy, mass 0; collision cylinder length=0.00 radius=0.0; visual cylinder length=0.00 radius=0.0
- added link torso_laser, mass 0.5; collision box size=0.05 0.065 0.12; visual box size=0.05 0.065 0.12
- added link torso_lasertop, mass 0.01; collision box size=0.05 0.065 0.01; visual box size=0.05 0.065 0.01
Joints:
- added joint torso_dummy_joint: type fixed, parent torso, child torso_dummy, origin xyz=-0.0994 0.0 0.075 rpy=0.0 -1.57 0.0, axis 0 1 0, limit lower=-0.7809 upper=1.5708 effort=13.4 velocity=1.0
- added joint torso_laser_joint: type fixed, parent torso_dummy, child torso_laser, origin xyz=0.0 0.0 0.0 rpy=0.0 0.0 -0.05, axis 0 1 0, limit lower=-0.7809 upper=1.5708 effort=13.4 velocity=1.0
- added joint torso_lasertop_joint: type fixed, parent torso_laser, child torso_lasertop

File: urdf/xacro/amigo.urdf.xacro (robot description, xacro)
@@ -15,6 +15,7 @@
 <!--extra body visuals-->
 <include filename="$(find amigo_description)/urdf/xacro/body_extra_visuals/body_extra.urdf.xacro" />
-<!--========BUILD LASER======-->
+<!--========BUILD LASERS======-->
 <include filename="$(find amigo_description)/urdf/xacro/laser/laser.urdf.xacro" />
+<include filename="$(find amigo_description)/urdf/xacro/laser/torso_laser.urdf.xacro" />
 <!--========BUILD HEAD======-->
 <include filename="$(find amigo_description)/urdf/xacro/head/head.urdf.xacro" />

File: urdf/xacro/gazebo.urdf.xacro (robot description, xacro)
@@ -177,4 +177,38 @@
       </sensor>
 </gazebo>
+<gazebo reference="torso_laser">
+      <sensor name='torso_ray_sensor' type='ray'>
+        <update_rate>100.000000</update_rate>
+        <ray>
+          <scan>
+            <horizontal>
+              <samples>918</samples>
+              <resolution>1.000000</resolution>
+              <min_angle>-2.0027654171</min_angle>
+              <max_angle>1.99840199947</max_angle>
+            </horizontal>
+            <vertical>
+              <samples>1</samples>
+              <min_angle>0.000000</min_angle>
+              <max_angle>0.000000</max_angle>
+            </vertical>
+          </scan>
+          <range>
+            <min>0.05</min>
+            <max>60.0</max>
+            <resolution>0.010000</resolution>
+          </range>
+        </ray>
+        <plugin name='torso_ros_ray_sensor_controller' filename='libLaserPlugin.so'>
+          <gaussianNoise>0.005</gaussianNoise>
+          <alwaysOn>1</alwaysOn>
+          <updateRate>40</updateRate>
+          <topicName>base_front_laser</topicName>
+          <node_namespace>base</node_namespace>
+          <frameName>base_laser</frameName>
+        </plugin>
+        <pose>0 0 0 0 0 0</pose>
+      </sensor>
+</gazebo>
 <gazebo reference="neck_tilt">
       <sensor name='openni_camera' type='depth'>

Commit message: Fixed finger joint limits
git-svn-id: https://roboticssrv.wtb.tue.nl/svn/ros/code/tue-ros-pkg/trunk/amigo_common/amigo_description@18447 3a3c2cfb-d3b9-409e-9e75-db8fcdbcaac6

File: urdf/amigo.urdf (robot description, URDF)
Before this commit: robot amigo, 75 links, 74 joints
Joints:
- joint finger1_joint_left: limit lower=-1.57 upper=1.57 effort=3 velocity=1.0 -> lower=0.2 upper=1 effort=3 velocity=1.0
- joint finger1_joint_right: limit lower=-1.57 upper=1.57 effort=3 velocity=1.0 -> lower=0.2 upper=1 effort=3 velocity=1.0
- joint finger1_tip_joint_left: limit lower=-1.57 upper=1.57 effort=3 velocity=1.0 -> lower=-0.6 upper=-0.2 effort=3 velocity=1.0
- joint finger1_tip_joint_right: limit lower=-1.57 upper=1.57 effort=3 velocity=1.0 -> lower=-0.6 upper=-0.2 effort=3 velocity=1.0
- joint finger2_joint_left: limit lower=-1.57 upper=1.57 effort=3 velocity=1.0 -> lower=0.2 upper=1 effort=3 velocity=1.0
- joint finger2_joint_right: limit lower=-1.57 upper=1.57 effort=3 velocity=1.0 -> lower=0.2 upper=1 effort=3 velocity=1.0
- joint finger2_tip_joint_left: limit lower=-1.57 upper=1.57 effort=3 velocity=1.0 -> lower=-0.6 upper=-0.2 effort=3 velocity=1.0
- joint finger2_tip_joint_right: limit lower=-1.57 upper=1.57 effort=3 velocity=1.0 -> lower=-0.6 upper=-0.2 effort=3 velocity=1.0

File: urdf/amigo_old.urdf (robot description, URDF)
Before this commit: robot amigo, 75 links, 74 joints
Joints:
- joint finger1_joint_left: limit lower=-1.57 upper=1.57 effort=3 velocity=1.0 -> lower=0.2 upper=1 effort=3 velocity=1.0
- joint finger1_joint_right: limit lower=-1.57 upper=1.57 effort=3 velocity=1.0 -> lower=0.2 upper=1 effort=3 velocity=1.0
- joint finger1_tip_joint_left: limit lower=-1.57 upper=1.57 effort=3 velocity=1.0 -> lower=-0.6 upper=-0.2 effort=3 velocity=1.0
- joint finger1_tip_joint_right: limit lower=-1.57 upper=1.57 effort=3 velocity=1.0 -> lower=-0.6 upper=-0.2 effort=3 velocity=1.0
- joint finger2_joint_left: limit lower=-1.57 upper=1.57 effort=3 velocity=1.0 -> lower=0.2 upper=1 effort=3 velocity=1.0
- joint finger2_joint_right: limit lower=-1.57 upper=1.57 effort=3 velocity=1.0 -> lower=0.2 upper=1 effort=3 velocity=1.0
- joint finger2_tip_joint_left: limit lower=-1.57 upper=1.57 effort=3 velocity=1.0 -> lower=-0.6 upper=-0.2 effort=3 velocity=1.0
- joint finger2_tip_joint_right: limit lower=-1.57 upper=1.57 effort=3 velocity=1.0 -> lower=-0.6 upper=-0.2 effort=3 velocity=1.0

File: urdf/xacro/arms/arm.urdf.xacro (robot description, xacro)
@@ -205,5 +205,5 @@
    <dynamics damping="0.5" friction="1.0"/>
    <axis xyz="1 0 0"/>
-   <limit effort="3" velocity="1.0" lower="-1.57" upper="1.57"/>
+   <limit effort="3" velocity="1.0" lower="0.2" upper="1"/>
 </xacro:my_joint>
 <joint name="finger1_phalanx_joint_${whichside}" type="fixed">
@@ -216,5 +216,5 @@
    <dynamics damping="0.5" friction="1.0"/>
    <axis xyz="1 0 0"/>
-   <limit effort="3" velocity="1.0" lower="-1.57" upper="1.57"/>
+   <limit effort="3" velocity="1.0" lower="-0.6" upper="-0.2"/>
 </xacro:my_joint>
 <joint name="finger1_tip_phalanx_joint_${whichside}" type="fixed">
@@ -227,5 +227,5 @@
    <dynamics damping="0.5" friction="1.0"/>
    <axis xyz="-1 0 0"/>
-   <limit effort="3" velocity="1.0" lower="-1.57" upper="1.57"/>
+   <limit effort="3" velocity="1.0" lower="0.2" upper="1"/>
 </xacro:my_joint>
 <joint name="finger2_phalanx_joint_${whichside}" type="fixed">
@@ -238,5 +238,5 @@
    <dynamics damping="0.5" friction="1.0"/>
    <axis xyz="-1 0 0"/>
-   <limit effort="3" velocity="1.0" lower="-1.57" upper="1.57"/>
+   <limit effort="3" velocity="1.0" lower="-0.6" upper="-0.2"/>
 </xacro:my_joint>
 <joint name="finger2_tip_phalanx_joint_${whichside}" type="fixed">

File: urdf/xacro/gazebo.urdf.xacro (robot description, xacro)
@@ -251,4 +251,14 @@
         <odomTopic>odom</odomTopic>
     </plugin>
+    <plugin name="left_gripper_controller" filename="libAmigoGripperController.so">
+		<side>left</side>
+		<referenceTopic>/amigo/left_gripper/references</referenceTopic>
+		<measurementTopic>/amigo/left_gripper/measurements</measurementTopic>
+    </plugin>
+    <plugin name="right_gripper_controller" filename="libAmigoGripperController.so">
+		<side>right</side>
+		<referenceTopic>/amigo/right_gripper/references</referenceTopic>
+		<measurementTopic>/amigo/right_gripper/measurements</measurementTopic>
+    </plugin>
 </gazebo>
 </robot>

Commit message: Updated urdf models with correct joint limits neck
git-svn-id: https://roboticssrv.wtb.tue.nl/svn/ros/code/tue-ros-pkg/trunk/amigo_common/amigo_description@18923 3a3c2cfb-d3b9-409e-9e75-db8fcdbcaac6

File: urdf/amigo.urdf (robot description, URDF)
Before this commit: robot amigo, 75 links, 74 joints
Joints:
- joint neck_tilt_joint: limit lower=-2.0 upper=2.0 effort=13.4 velocity=1.0 -> lower=-0.5 upper=0.88 effort=13.4 velocity=1.0

File: urdf/amigo_old.urdf (robot description, URDF)
Before this commit: robot amigo, 75 links, 74 joints
Joints:
- joint neck_tilt_joint: limit lower=-2.0 upper=2.0 effort=13.4 velocity=1.0 -> lower=-0.5 upper=0.88 effort=13.4 velocity=1.0

File: urdf/xacro/head/head.urdf.xacro (robot description, xacro)
@@ -56,5 +56,5 @@
    <dynamics damping="0.1" friction="0.0"/>
    <axis xyz="0 1 0"/>
-   <limit effort="13.4" velocity="1.0" lower="-2.0" upper="2.0" />
+   <limit effort="13.4" velocity="1.0" lower="-0.5" upper="0.88" />
 </xacro:my_joint>
 </robot>

Commit message: Fixed torso joint lower limit
git-svn-id: https://roboticssrv.wtb.tue.nl/svn/ros/code/tue-ros-pkg/trunk/amigo_common/amigo_description@20612 3a3c2cfb-d3b9-409e-9e75-db8fcdbcaac6

File: urdf/amigo.urdf (robot description, URDF)
Before this commit: robot amigo, 75 links, 74 joints
Joints:
- joint torso_joint: limit lower=0.0 upper=0.41 effort=1000 velocity=10.0 -> lower=0.075 upper=0.41 effort=1000 velocity=10.0

File: urdf/xacro/body/body.urdf.xacro (robot description, xacro)
@@ -40,5 +40,5 @@
   <origin xyz="0.0 0.0 0.58" rpy="3.14159265 -1.5708 0"/>
   <dynamics damping="3" friction="0.0"/> <!--*-->
-  <limit effort="1000" velocity="10.0" lower="0.0" upper="0.41" /> <!--*-->
+  <limit effort="1000" velocity="10.0" lower="0.075" upper="0.41" /> <!--*-->
 </joint>
 <joint name="base_link_joint" type="fixed">

Commit message: Updated kinect topic
git-svn-id: https://roboticssrv.wtb.tue.nl/svn/ros/code/tue-ros-pkg/trunk/amigo_common/amigo_description@22466 3a3c2cfb-d3b9-409e-9e75-db8fcdbcaac6

File: urdf/amigo.urdf (robot description, URDF)
Before this commit: robot amigo, 75 links, 74 joints
Joints:
- joint top_kinect/base_kinect_joint: origin xyz=0.07 0 0.07 rpy=0 0 0 -> xyz=0.07 0.05 0.10 rpy=0 0.01 0.015

File: urdf/xacro/gazebo.urdf.xacro (robot description, xacro)
@@ -139,5 +139,5 @@
           <depthImageTopicName>depth_registered/image</depthImageTopicName>
           <depthImageCameraInfoTopicName>depth/camera_info</depthImageCameraInfoTopicName>
-          <pointCloudTopicName>rgb/points</pointCloudTopicName>
+          <pointCloudTopicName>depth_registered/points</pointCloudTopicName>
           <frameName>base_kinect/openni_depth_optical_frame</frameName>
         </plugin>
@@ -234,5 +234,5 @@
           <depthImageTopicName>depth_registered/image</depthImageTopicName>
           <depthImageCameraInfoTopicName>depth/camera_info</depthImageCameraInfoTopicName>
-          <pointCloudTopicName>rgb/points</pointCloudTopicName>
+          <pointCloudTopicName>depth_registered/points</pointCloudTopicName>
           <frameName>top_kinect/openni_depth_optical_frame</frameName>
         </plugin>

Commit message: Updated urdf and sdf files
git-svn-id: https://roboticssrv.wtb.tue.nl/svn/ros/trunk/amigo_common/amigo_description@24428 3a3c2cfb-d3b9-409e-9e75-db8fcdbcaac6

File: urdf/amigo.urdf (robot description, URDF)
Before this commit: robot amigo, 75 links, 74 joints
Joints:
- joint head_mount_joint: origin xyz=0.097 0.0 0.0 rpy=  0.0 0.0 0.0 -> xyz=0.11 0.0 0.0 rpy=  0.0 0.0 0.0
- joint top_kinect/base_kinect_joint: origin xyz=0.07 0.05 0.10 rpy=0 0.01 0.015 -> xyz=0.07 0.05 0.10 rpy=0.02 0.01 0.015

Commit message: Updated URDF model
git-svn-id: https://roboticssrv.wtb.tue.nl/svn/ros/trunk/amigo_common/amigo_description@24663 3a3c2cfb-d3b9-409e-9e75-db8fcdbcaac6

File: urdf/amigo.urdf (robot description, URDF)
Before this commit: robot amigo, 75 links, 74 joints
Joints:
- joint base_laser_joint: origin xyz=0.31 0.0 0.185 rpy=0 0 0 -> xyz=0.3239 0.0 0.24 rpy=0 0 0.015
- joint head_mount_joint: origin xyz=0.11 0.0 0.0 rpy=  0.0 0.0 0.0 -> xyz=0.11 0.0 0.0426 rpy=0.0 0.0 0.0
- joint neck_pan_joint: origin xyz=0.0 0.0 0.0 rpy=3.14 -1.5708 0.0 -> xyz=0.0 0.0 0.0 rpy=3.1415 -1.5708 0.0
- joint neck_tilt_joint: origin xyz=0.0 0.0 0.0445 rpy=0.0 0.0 0.0 -> xyz=0.0 0.0 0.0445 rpy=0.0 0.015 0.0
- joint top_kinect/base_kinect_joint: origin xyz=0.07 0.05 0.10 rpy=0.02 0.01 0.015 -> xyz=0.035 0.0 0.10 rpy=0.0 0.0 0.025
- joint top_kinect/kinect_depth_joint: origin xyz=0 0.018 0 rpy=0 0 0 -> xyz=0 0.0125 0 rpy=0 0 0
- joint top_kinect/kinect_rgb_joint: origin xyz=0 -0.005 0 rpy=0 0 0 -> xyz=0 -0.0125 0 rpy=0 0 0

File: urdf/xacro/head/head.urdf.xacro (robot description, xacro)
@@ -17,5 +17,5 @@
   <child link="head_mount"/>
   <axis xyz="0 0 1"/>
-  <origin xyz="0.11 0.0 0.0" rpy="  0.0 0.0 0.0"/>
+  <origin xyz="0.11 0.0 0.0426" rpy="0.0 0.0 0.0"/>
 </joint>
 <!-- the link that represents the panning part of the neck, is below neck_tilt -->
@@ -37,5 +37,5 @@
  <my_link_texturedmesh name="head" mass="0" texture="white">
    <origin xyz="0 0 0.041" rpy="0 0 0"/>
-   <origin xyz="0.0 0.0 0.141" rpy="0 0 -1.5708"/>
+   <origin xyz="0.0 0.0 0.141" rpy="0 0 -1.5708"/><!-- Updated for visual purpose -->
    <inertia ixx="0"  ixy="0"  ixz="0" iyy="0" iyz="0" izz="0" />
    <mesh filename="package://amigo_description/media/meshes/headtextured.dae" scale="0.0004 0.0004 0.0004"/>
@@ -47,5 +47,5 @@
 <!-- the tilt and pan joints-->
 <xacro:my_joint name="neck_pan_joint" type="revolute" parent="head_mount" child="neck_pan">
-   <origin xyz="0.0 0.0 0.0" rpy="3.14 -1.5708 0.0"/>
+   <origin xyz="0.0 0.0 0.0" rpy="3.1415 -1.5708 0.0"/>
    <dynamics damping="0.1" friction="0"/>
    <axis xyz="0 0 1"/>
@@ -53,5 +53,5 @@
 </xacro:my_joint>
 <xacro:my_joint name="neck_tilt_joint" type="revolute" parent="neck_pan" child="neck_tilt">
-   <origin xyz="0.0 0.0 0.0445" rpy="0.0 0.0 0.0"/>
+   <origin xyz="0.0 0.0 0.0445" rpy="0.0 0.015 0.0"/>
    <dynamics damping="0.1" friction="0.0"/>
    <axis xyz="0 1 0"/>

File: urdf/xacro/kinect/top_kinect.urdf.xacro (robot description, xacro)
@@ -6,5 +6,6 @@
   <property name="M_PI" value="3.14159"/>
   <joint name="top_kinect/base_kinect_joint" type="fixed">
-    <origin xyz="0.07 0.05 0.10" rpy="0.02 0.01 0.015" /> <!-- THESE VALUES ARE ROUGH ESTIMATES!! -->
+    <origin xyz="0.035 0.0 0.10" rpy="0.0 0.0 0.025" /> <!-- THESE VALUES ARE ROUGH ESTIMATES!! -->
+    <origin xyz="0.035 0.0 0.10" rpy="0.0 0.0 0.025" /> <!-- THESE VALUES ARE ROUGH ESTIMATES!! -->
     <parent link="head" />
     <child link="top_kinect/openni_camera" />
@@ -34,5 +35,5 @@
   </link>
   <joint name="top_kinect/kinect_depth_joint" type="fixed">
-    <origin xyz="0 0.018 0" rpy="0 0 0" />
+    <origin xyz="0 0.0125 0" rpy="0 0 0" />
     <parent link="top_kinect/openni_camera" />
     <child link="top_kinect/openni_depth_frame" />
@@ -62,5 +63,5 @@
   </link>
   <joint name="top_kinect/kinect_rgb_joint" type="fixed">
-    <origin xyz="0 -0.005 0" rpy="0 0 0" />
+    <origin xyz="0 -0.0125 0" rpy="0 0 0" />
     <parent link="top_kinect/openni_camera" />
     <child link="top_kinect/openni_rgb_frame" />

File: urdf/xacro/laser/laser.urdf.xacro (robot description, xacro)
@@ -12,5 +12,5 @@
 </xacro:my_link>
 <xacro:my_joint name="base_laser_joint" type="fixed" parent="base" child="base_laser">
-   <origin xyz="0.31 0.0 0.185" rpy="0 0 0"/>
+   <origin xyz="0.3239 0.0 0.24" rpy="0 0 0.015"/><!-- (plateWidth + plateEdge->centerOfPole + centerOfPole->centerOfLaser = 30+1.65+0.74. Height = 0.295 - 0.055 = 0.24 (base height = 0.055)-->
    <dynamics damping="0.1" friction="0"/>
    <axis xyz="0 1 0"/>

Commit message: new urdf model with back laser
git-svn-id: https://roboticssrv.wtb.tue.nl/svn/ros/trunk/amigo_common/amigo_description@24995 3a3c2cfb-d3b9-409e-9e75-db8fcdbcaac6

File: urdf/amigo.urdf (robot description, URDF)
Before this commit: robot amigo, 75 links, 74 joints
Links:
- added link back_laser, mass 0.5; collision box size=0.05 0.065 0.12; visual box size=0.05 0.065 0.12
- added link back_lasertop, mass 0.01; collision box size=0.05 0.065 0.01; visual box size=0.05 0.065 0.01
Joints:
- added joint back_laser_joint: type fixed, parent base, child back_laser, origin xyz=-0.275 0.0 0.235 rpy=0 0 3.11, axis 0 1 0, limit lower=-0.7809 upper=1.5708 effort=13.4 velocity=1.0
- added joint back_lasertop_joint: type fixed, parent back_laser, child back_lasertop

File: urdf/xacro/amigo.urdf.xacro (robot description, xacro)
@@ -18,4 +18,5 @@
 <include filename="$(find amigo_description)/urdf/xacro/laser/laser.urdf.xacro" />
 <include filename="$(find amigo_description)/urdf/xacro/laser/torso_laser.urdf.xacro" />
+<include filename="$(find amigo_description)/urdf/xacro/laser/back_laser.urdf.xacro" />
 <!--========BUILD HEAD======-->
 <include filename="$(find amigo_description)/urdf/xacro/head/head.urdf.xacro" />

File: urdf/xacro/laser/back_laser.urdf.xacro (robot description, xacro)
@@ -5,5 +5,4 @@
    <review status="unreviewed" notes=""/>
 <!--the laser at the back of the base of the robot -->
-<!--To Do: check exact dimensions -->
 <xacro:my_link name="back_laser" mass="0.5" color="Black">
    <box size="0.05 0.065 0.12" />
@@ -13,5 +12,5 @@
 </xacro:my_link>
 <xacro:my_joint name="back_laser_joint" type="fixed" parent="base" child="back_laser">
-   <origin xyz="-0.3239 0.0 0.235" rpy="0 0 3.14"/><!-- (plateWidth + plateEdge->centerOfPole + centerOfPole->centerOfLaser = 30+1.65+0.74. Height = 0.295 - 0.055 = 0.24 (base height = 0.055)-->
+   <origin xyz="-0.275 0.0 0.235" rpy="0 0 3.11"/><!-- (plateWidth + plateEdge->centerOfPole + centerOfPole->centerOfLaser = 30+1.65+0.74. Height = 0.295 - 0.055 = 0.24 (base height = 0.055)-->
    <dynamics damping="0.1" friction="0"/>
    <axis xyz="0 1 0"/>
@@ -19,5 +18,5 @@
 </xacro:my_joint>
 <!--the orange top of the laser-->
-<xacro:my_link_textured name="lasertop" mass="0.01" texture="orange">
+<xacro:my_link_textured name="back_lasertop" mass="0.01" texture="orange">
    <box size="0.05 0.065 0.01" />
    <origin xyz="0.0 0.0 0.0" rpy="0 0 0"/>
@@ -25,7 +24,7 @@
    <inertia ixx="0.0001"  ixy="0"  ixz="0" iyy="0.0001" iyz="0" izz="0.0001" />
 </xacro:my_link_textured>
-<joint name="lasertop_joint" type="fixed">
+<joint name="back_lasertop_joint" type="fixed">
     <parent link="back_laser"/>
-    <child link="lasertop"/>
+    <child link="back_lasertop"/>
 </joint>
 </robot>

Commit message: Updated tf for camera

File: urdf/amigo.urdf (robot description, URDF)
Before this commit: robot amigo, 77 links, 76 joints
Joints:
- joint torso_slider_joint: origin xyz=0.135 0.0 0.0 rpy=0 0 0 -> xyz=0.1 0.0 0.0 rpy=0 0 0

File: urdf/xacro/body/body.urdf.xacro (robot description, xacro)
@@ -52,5 +52,5 @@
   <child link="torso"/>
   <axis xyz="1 0 0"/>
-  <origin xyz="0.135 0.0 0.0" rpy="0 0 0"/>
+  <origin xyz="0.1 0.0 0.0" rpy="0 0 0"/>
 </joint>
 </robot>

Commit message: making sure joint limits urdf model match those in ops files in amigo_bringup

File: urdf/amigo.urdf (robot description, URDF)
Before this commit: robot amigo, 77 links, 76 joints
Joints:
- joint torso_dummy_joint: origin xyz=-0.0994 0.0 0.075 rpy=0.0 -1.57 0.0 -> xyz=-0.0994 0.0 0.09 rpy=0.0 -1.57 0.0
- joint torso_joint: limit lower=0.075 upper=0.41 effort=1000 velocity=10.0 -> lower=0.09 upper=0.4 effort=1000 velocity=10.0

Commit message: Changing urdf via xacro this time... And torso max set to 0.41

File: urdf/amigo.urdf (robot description, URDF)
Before this commit: robot amigo, 77 links, 76 joints
Joints:
- joint torso_dummy_joint: origin xyz=-0.0994 0.0 0.09 rpy=0.0 -1.57 0.0 -> xyz=-0.0994 0.0 0.075 rpy=0.0 -1.57 0.0
- joint torso_joint: limit lower=0.09 upper=0.4 effort=1000 velocity=10.0 -> lower=0.09 upper=0.41 effort=1000 velocity=10.0

File: urdf/xacro/body/body.urdf.xacro (robot description, xacro)
@@ -40,5 +40,5 @@
   <origin xyz="0.0 0.0 0.58" rpy="3.14159265 -1.5708 0"/>
   <dynamics damping="3" friction="0.0"/> <!--*-->
-  <limit effort="1000" velocity="10.0" lower="0.075" upper="0.41" /> <!--*-->
+  <limit effort="1000" velocity="10.0" lower="0.09" upper="0.41" /> <!--*-->
 </joint>
 <joint name="base_link_joint" type="fixed">
