Commit message: Modified velocities to stroke with ops files

File: urdf/amigo.urdf (robot description, URDF)
Before this commit: robot amigo, 77 links, 76 joints
Joints:
- joint elbow_pitch_joint_left: limit lower=0.0 upper=2.23 effort=4.5 velocity=1.0 -> lower=0.0 upper=2.23 effort=4.5 velocity=0.8
- joint elbow_pitch_joint_right: limit lower=0.0 upper=2.23 effort=4.5 velocity=1.0 -> lower=0.0 upper=2.23 effort=4.5 velocity=0.8
- joint elbow_roll_joint_left: limit lower=-1.83 upper=1.83 effort=4.5 velocity=1.0 -> lower=-1.83 upper=1.83 effort=4.5 velocity=0.8
- joint elbow_roll_joint_right: limit lower=-1.83 upper=1.83 effort=4.5 velocity=1.0 -> lower=-1.83 upper=1.83 effort=4.5 velocity=0.8
- joint shoulder_pitch_joint_left: limit lower=-1.57 upper=1.57 effort=13.4 velocity=1.0 -> lower=-1.57 upper=1.57 effort=13.4 velocity=0.4
- joint shoulder_pitch_joint_right: limit lower=-1.57 upper=1.57 effort=13.4 velocity=1.0 -> lower=-1.57 upper=1.57 effort=13.4 velocity=0.4
- joint shoulder_roll_joint_left: limit lower=-1.57 upper=1.57 effort=9.8 velocity=1.0 -> lower=-1.57 upper=1.57 effort=9.8 velocity=0.6
- joint shoulder_roll_joint_right: limit lower=-1.57 upper=1.57 effort=9.8 velocity=1.0 -> lower=-1.57 upper=1.57 effort=9.8 velocity=0.6
- joint shoulder_yaw_joint_left: limit lower=-1.57 upper=0.0 effort=13.4 velocity=1.0 -> lower=-1.57 upper=0.0 effort=13.4 velocity=0.4
- joint shoulder_yaw_joint_right: limit lower=-1.57 upper=0.0 effort=13.4 velocity=1.0 -> lower=-1.57 upper=0.0 effort=13.4 velocity=0.4

File: urdf/xacro/arms/arm.urdf.xacro (robot description, xacro)
@@ -163,5 +163,5 @@
    <dynamics damping="4.0" friction="4.87"/>
    <axis xyz="${rollsign}1 0 0"/>
-   <limit effort="13.4" velocity="1.0" lower="-1.57" upper="0.0" />
+   <limit effort="13.4" velocity="0.4" lower="-1.57" upper="0.0" />
 </xacro:my_joint>
 <xacro:my_joint name="shoulder_pitch_joint_${whichside}" type="revolute" parent="shoulder_link1_${whichside}" child="shoulder_link2_${whichside}">
@@ -169,5 +169,5 @@
    <dynamics damping="4.0" friction="6.06"/>
    <axis xyz="0 -1 0"/>
-   <limit effort="13.4" velocity="1.0" lower="-1.57" upper="1.57" />
+   <limit effort="13.4" velocity="0.4" lower="-1.57" upper="1.57" />
 </xacro:my_joint>
 <xacro:my_joint name="shoulder_roll_joint_${whichside}" type="revolute" parent="shoulder_link2_${whichside}" child="upper_arm_${whichside}">
@@ -175,5 +175,5 @@
    <dynamics damping="3.8" friction="2.216"/>
    <axis xyz="0 ${sidesign} 0"/>
-   <limit effort="9.8" velocity="1.0" lower="-1.57" upper="1.57"/>
+   <limit effort="9.8" velocity="0.6" lower="-1.57" upper="1.57"/>
 </xacro:my_joint>
 <xacro:my_joint name="elbow_pitch_joint_${whichside}" type="revolute" parent="upper_arm_${whichside}" child="elbow_link4_${whichside}">
@@ -181,5 +181,5 @@
    <dynamics damping="3" friction="1.18"/>
    <axis xyz="0 -1 0"/>
-   <limit effort="4.5" velocity="1.0" lower="0.0" upper="2.23" />
+   <limit effort="4.5" velocity="0.8" lower="0.0" upper="2.23" />
 </xacro:my_joint>
 <xacro:my_joint name="elbow_roll_joint_${whichside}" type="revolute" parent="elbow_link4_${whichside}" child="fore_arm_${whichside}">
@@ -187,5 +187,5 @@
    <dynamics damping="3.5" friction="1.35"/>
    <axis xyz="0 ${sidesign} 0"/>
-   <limit effort="4.5" velocity="1.0" lower="-1.83" upper="1.83"/>
+   <limit effort="4.5" velocity="0.8" lower="-1.83" upper="1.83"/>
 </xacro:my_joint>
 <xacro:my_joint name="wrist_pitch_joint_${whichside}" type="revolute" parent="fore_arm_${whichside}" child="wrist_link6_${whichside}">

Commit message: Working on moveit for manip

File: urdf/amigo.urdf (robot description, URDF)
Before this commit: robot amigo, 77 links, 76 joints
Links:
- link base_link: mass 0 -> None; geometry 

File: urdf/xacro/body/body.urdf.xacro (robot description, xacro)
@@ -27,10 +27,6 @@
 </xacro:my_link_texturedmesh>
 <!--the root of the tf-tree, because it serves only this function it has no visuals-->
-<xacro:my_link name="base_link" mass="0" color="Red">
-   <cylinder radius="0.0" length="0.00" />
-   <origin xyz="0.0 0.0 0.0" rpy="0 0 0"/>
-   <origin xyz="0.0 0.0 0.0" rpy="0 0 0" />
-   <inertia ixx="0"  ixy="0"  ixz="0" iyy="0" iyz="0" izz="0" />
-</xacro:my_link>
+<link name="base_link">
+</link>
 <!-- joints start here -->
 <joint name="torso_joint" type="prismatic">

Commit message: Made limits consistent with ops files

File: urdf/amigo.urdf (robot description, URDF)
Before this commit: robot amigo, 77 links, 76 joints
Joints:
- joint elbow_pitch_joint_left: limit lower=0.0 upper=2.23 effort=4.5 velocity=0.8 -> lower=0.0 upper=2.23 effort=0.5 velocity=0.8
- joint elbow_pitch_joint_right: limit lower=0.0 upper=2.23 effort=4.5 velocity=0.8 -> lower=0.0 upper=2.23 effort=0.5 velocity=0.8
- joint elbow_roll_joint_left: limit lower=-1.83 upper=1.83 effort=4.5 velocity=0.8 -> lower=-1.83 upper=1.83 effort=0.5 velocity=0.8
- joint elbow_roll_joint_right: limit lower=-1.83 upper=1.83 effort=4.5 velocity=0.8 -> lower=-1.83 upper=1.83 effort=0.5 velocity=0.8
- joint shoulder_pitch_joint_left: limit lower=-1.57 upper=1.57 effort=13.4 velocity=0.4 -> lower=-1.57 upper=1.57 effort=0.2 velocity=0.4
- joint shoulder_pitch_joint_right: limit lower=-1.57 upper=1.57 effort=13.4 velocity=0.4 -> lower=-1.57 upper=1.57 effort=0.2 velocity=0.4
- joint shoulder_roll_joint_left: limit lower=-1.57 upper=1.57 effort=9.8 velocity=0.6 -> lower=-1.57 upper=1.57 effort=0.3 velocity=0.6
- joint shoulder_roll_joint_right: limit lower=-1.57 upper=1.57 effort=9.8 velocity=0.6 -> lower=-1.57 upper=1.57 effort=0.3 velocity=0.6
- joint shoulder_yaw_joint_left: limit lower=-1.57 upper=0.0 effort=13.4 velocity=0.4 -> lower=-1.57 upper=0.0 effort=0.2 velocity=0.4
- joint shoulder_yaw_joint_right: limit lower=-1.57 upper=0.0 effort=13.4 velocity=0.4 -> lower=-1.57 upper=0.0 effort=0.2 velocity=0.4
- joint torso_joint: limit lower=0.09 upper=0.41 effort=1000 velocity=10.0 -> lower=0.075 upper=0.4 effort=0.1 velocity=0.07
- joint wrist_pitch_joint_left: limit lower=-0.95 upper=0.95 effort=1 velocity=1.0 -> lower=-0.95 upper=0.95 effort=0.5 velocity=1.0
- joint wrist_pitch_joint_right: limit lower=-0.95 upper=0.95 effort=1 velocity=1.0 -> lower=-0.95 upper=0.95 effort=0.5 velocity=1.0
- joint wrist_yaw_joint_left: limit lower=-0.61 upper=0.61 effort=1 velocity=1.0 -> lower=-0.61 upper=0.61 effort=0.5 velocity=1.0
- joint wrist_yaw_joint_right: limit lower=-0.61 upper=0.61 effort=1 velocity=1.0 -> lower=-0.61 upper=0.61 effort=0.5 velocity=1.0

File: urdf/xacro/arms/arm.urdf.xacro (robot description, xacro)
@@ -163,5 +163,5 @@
    <dynamics damping="4.0" friction="4.87"/>
    <axis xyz="${rollsign}1 0 0"/>
-   <limit effort="13.4" velocity="0.4" lower="-1.57" upper="0.0" />
+   <limit effort="0.2" velocity="0.4" lower="-1.57" upper="0.0" />
 </xacro:my_joint>
 <xacro:my_joint name="shoulder_pitch_joint_${whichside}" type="revolute" parent="shoulder_link1_${whichside}" child="shoulder_link2_${whichside}">
@@ -169,5 +169,5 @@
    <dynamics damping="4.0" friction="6.06"/>
    <axis xyz="0 -1 0"/>
-   <limit effort="13.4" velocity="0.4" lower="-1.57" upper="1.57" />
+   <limit effort="0.2" velocity="0.4" lower="-1.57" upper="1.57" />
 </xacro:my_joint>
 <xacro:my_joint name="shoulder_roll_joint_${whichside}" type="revolute" parent="shoulder_link2_${whichside}" child="upper_arm_${whichside}">
@@ -175,5 +175,5 @@
    <dynamics damping="3.8" friction="2.216"/>
    <axis xyz="0 ${sidesign} 0"/>
-   <limit effort="9.8" velocity="0.6" lower="-1.57" upper="1.57"/>
+   <limit effort="0.3" velocity="0.6" lower="-1.57" upper="1.57"/>
 </xacro:my_joint>
 <xacro:my_joint name="elbow_pitch_joint_${whichside}" type="revolute" parent="upper_arm_${whichside}" child="elbow_link4_${whichside}">
@@ -181,5 +181,5 @@
    <dynamics damping="3" friction="1.18"/>
    <axis xyz="0 -1 0"/>
-   <limit effort="4.5" velocity="0.8" lower="0.0" upper="2.23" />
+   <limit effort="0.5" velocity="0.8" lower="0.0" upper="2.23" />
 </xacro:my_joint>
 <xacro:my_joint name="elbow_roll_joint_${whichside}" type="revolute" parent="elbow_link4_${whichside}" child="fore_arm_${whichside}">
@@ -187,5 +187,5 @@
    <dynamics damping="3.5" friction="1.35"/>
    <axis xyz="0 ${sidesign} 0"/>
-   <limit effort="4.5" velocity="0.8" lower="-1.83" upper="1.83"/>
+   <limit effort="0.5" velocity="0.8" lower="-1.83" upper="1.83"/>
 </xacro:my_joint>
 <xacro:my_joint name="wrist_pitch_joint_${whichside}" type="revolute" parent="fore_arm_${whichside}" child="wrist_link6_${whichside}">
@@ -193,5 +193,5 @@
    <dynamics damping="0.35" friction="0.63"/>
    <axis xyz="0 -1 0"/>
-   <limit effort="1" velocity="1.0" lower="-0.95" upper="0.95"/>
+   <limit effort="0.5" velocity="1.0" lower="-0.95" upper="0.95"/>
 </xacro:my_joint>
 <xacro:my_joint name="wrist_yaw_joint_${whichside}" type="revolute" parent="wrist_link6_${whichside}" child="hand_${whichside}">
@@ -199,5 +199,5 @@
    <dynamics damping="0.3" friction="0.68"/>
    <axis xyz="0 0 ${sidesign}1"/>
-   <limit effort="1" velocity="1.0" lower="-0.61" upper="0.61"/>
+   <limit effort="0.5" velocity="1.0" lower="-0.61" upper="0.61"/>
 </xacro:my_joint>
 <xacro:my_joint name="finger1_joint_${whichside}" type="revolute" parent="hand_${whichside}" child="finger1_${whichside}">

File: urdf/xacro/body/body.urdf.xacro (robot description, xacro)
@@ -40,5 +40,5 @@
   <origin xyz="0.0 0.0 0.58" rpy="3.14159265 -1.5708 0"/>
   <dynamics damping="3" friction="0.0"/> <!--*-->
-  <limit effort="1000" velocity="10.0" lower="0.09" upper="0.41" /> <!--*-->
+  <limit effort="0.1" velocity="0.07" lower="0.075" upper="0.4" />
 </joint>
 <joint name="base_link_joint" type="fixed">

Commit message: Increased lower limit of spidle

File: urdf/amigo.urdf (robot description, URDF)
Before this commit: robot amigo, 77 links, 76 joints
Joints:
- joint torso_joint: limit lower=0.075 upper=0.4 effort=0.1 velocity=0.07 -> lower=0.09 upper=0.4 effort=0.1 velocity=0.07

File: urdf/xacro/body/body.urdf.xacro (robot description, xacro)
@@ -40,5 +40,5 @@
   <origin xyz="0.0 0.0 0.58" rpy="3.14159265 -1.5708 0"/>
   <dynamics damping="3" friction="0.0"/> <!--*-->
-  <limit effort="0.1" velocity="0.07" lower="0.075" upper="0.4" />
+  <limit effort="0.1" velocity="0.07" lower="0.09" upper="0.4" />
 </joint>
 <joint name="base_link_joint" type="fixed">

Commit message: Fixed prefixes again

File: urdf/amigo.urdf (robot description, URDF)
Before this commit: robot amigo, 77 links, 76 joints
Links:
- link amigo/base_link: mass 0 -> None; geometry 

File: urdf/xacro/body/body.urdf.xacro (robot description, xacro)
@@ -28,5 +28,5 @@
 </xacro:my_link_texturedmesh>
 <!--the root of the tf-tree, because it serves only this function it has no visuals-->
-<link name="base_link" type="planar">
+<link name="${prefix}base_link" type="planar">
    <cylinder radius="0.0" length="0.00" />
    <origin xyz="0.0 0.0 0.0" rpy="0 0 0"/>

File: urdf/xacro/kinect/base_kinect.urdf.xacro (robot description, xacro)
@@ -8,8 +8,8 @@
   <joint name="base_kinect/base_kinect_joint" type="fixed">
     <origin xyz="0.3 0 0.26" rpy="0 -0.07 0" /> <!-- THESE VALUES STILL HAVE TO BE CALIBRATED!! -->
-    <parent link="base" />
-    <child link="base_kinect/openni_camera" />
+    <parent link="${prefix}base" />
+    <child link="${prefix}base_kinect/openni_camera" />
   </joint>
-  <link name="base_kinect/openni_camera">
+  <link name="${prefix}base_kinect/openni_camera">
     <inertial>
       <mass value="0.01" />
@@ -38,8 +38,8 @@
   <joint name="base_kinect/kinect_depth_joint" type="fixed">
     <origin xyz="0 0.018 0" rpy="0 0 0" />
-    <parent link="base_kinect/openni_camera" />
-    <child link="base_kinect/openni_depth_frame" />
+    <parent link="${prefix}base_kinect/openni_camera" />
+    <child link="${prefix}base_kinect/openni_depth_frame" />
   </joint>
-  <link name="base_kinect/openni_depth_frame">
+  <link name="${prefix}base_kinect/openni_depth_frame">
     <inertial>
       <mass value="0.01" />
@@ -52,8 +52,8 @@
   <joint name="base_kinect/kinect_depth_optical_joint" type="fixed">
     <origin xyz="0 0 0" rpy="${-M_PI/2} 0 ${-M_PI/2}" />
-    <parent link="base_kinect/openni_depth_frame" />
-    <child link="base_kinect/openni_depth_optical_frame" />
+    <parent link="${prefix}base_kinect/openni_depth_frame" />
+    <child link="${prefix}base_kinect/openni_depth_optical_frame" />
   </joint>
-  <link name="base_kinect/openni_depth_optical_frame">
+  <link name="${prefix}base_kinect/openni_depth_optical_frame">
     <inertial>
       <mass value="0.001" />
@@ -66,8 +66,8 @@
   <joint name="base_kinect/kinect_rgb_joint" type="fixed">
     <origin xyz="0 -0.005 0" rpy="0 0 0" />
-    <parent link="base_kinect/openni_camera" />
-    <child link="base_kinect/openni_rgb_frame" />
+    <parent link="${prefix}base_kinect/openni_camera" />
+    <child link="${prefix}base_kinect/openni_rgb_frame" />
   </joint>
-  <link name="base_kinect/openni_rgb_frame">
+  <link name="${prefix}base_kinect/openni_rgb_frame">
     <inertial>
       <mass value="0.001" />
@@ -80,8 +80,8 @@
   <joint name="base_kinect/kinect_rgb_optical_joint" type="fixed">
     <origin xyz="0 0 0" rpy="${-M_PI/2} 0 ${-M_PI/2}" />
-    <parent link="base_kinect/openni_rgb_frame" />
-    <child link="base_kinect/openni_rgb_optical_frame" />
+    <parent link="${prefix}base_kinect/openni_rgb_frame" />
+    <child link="${prefix}base_kinect/openni_rgb_optical_frame" />
   </joint>
-  <link name="base_kinect/openni_rgb_optical_frame">
+  <link name="${prefix}base_kinect/openni_rgb_optical_frame">
     <inertial>
       <mass value="0.001" />

File: urdf/xacro/kinect/top_kinect.urdf.xacro (robot description, xacro)
@@ -9,8 +9,8 @@
     <origin xyz="0.035 0.0 0.10" rpy="0.0 0.0 0.025" /> <!-- THESE VALUES ARE ROUGH ESTIMATES!! -->
     <origin xyz="0.035 0.0 0.10" rpy="0.0 0.0 0.025" /> <!-- THESE VALUES ARE ROUGH ESTIMATES!! -->
-    <parent link="head" />
-    <child link="top_kinect/openni_camera" />
+    <parent link="${prefix}head" />
+    <child link="${prefix}top_kinect/openni_camera" />
   </joint>
-  <link name="top_kinect/openni_camera">
+  <link name="${prefix}top_kinect/openni_camera">
     <inertial>
       <mass value="0.01" />
@@ -37,8 +37,8 @@
   <joint name="top_kinect/kinect_depth_joint" type="fixed">
     <origin xyz="0 0.0125 0" rpy="0 0 0" />
-    <parent link="top_kinect/openni_camera" />
-    <child link="top_kinect/openni_depth_frame" />
+    <parent link="${prefix}top_kinect/openni_camera" />
+    <child link="${prefix}top_kinect/openni_depth_frame" />
   </joint>
-  <link name="top_kinect/openni_depth_frame">
+  <link name="${prefix}top_kinect/openni_depth_frame">
     <inertial>
       <mass value="0.01" />
@@ -51,8 +51,8 @@
   <joint name="top_kinect/kinect_depth_optical_joint" type="fixed">
     <origin xyz="0 0 0" rpy="${-M_PI/2} 0 ${-M_PI/2}" />
-    <parent link="top_kinect/openni_depth_frame" />
-    <child link="top_kinect/openni_depth_optical_frame" />
+    <parent link="${prefix}top_kinect/openni_depth_frame" />
+    <child link="${prefix}top_kinect/openni_depth_optical_frame" />
   </joint>
-  <link name="top_kinect/openni_depth_optical_frame">
+  <link name="${prefix}top_kinect/openni_depth_optical_frame">
     <inertial>
       <mass value="0.001" />
@@ -65,8 +65,8 @@
   <joint name="top_kinect/kinect_rgb_joint" type="fixed">
     <origin xyz="0 -0.0125 0" rpy="0 0 0" />
-    <parent link="top_kinect/openni_camera" />
-    <child link="top_kinect/openni_rgb_frame" />
+    <parent link="${prefix}top_kinect/openni_camera" />
+    <child link="${prefix}top_kinect/openni_rgb_frame" />
   </joint>
-  <link name="top_kinect/openni_rgb_frame">
+  <link name="${prefix}top_kinect/openni_rgb_frame">
     <inertial>
       <mass value="0.001" />
@@ -79,8 +79,8 @@
   <joint name="top_kinect/kinect_rgb_optical_joint" type="fixed">
     <origin xyz="0 0 0" rpy="${-M_PI/2} 0 ${-M_PI/2}" />
-    <parent link="top_kinect/openni_rgb_frame" />
-    <child link="top_kinect/openni_rgb_optical_frame" />
+    <parent link="${prefix}top_kinect/openni_rgb_frame" />
+    <child link="${prefix}top_kinect/openni_rgb_optical_frame" />
   </joint>
-  <link name="top_kinect/openni_rgb_optical_frame">
+  <link name="${prefix}top_kinect/openni_rgb_optical_frame">
     <inertial>
       <mass value="0.001" />
