Commit message: Minimal implementation to work under kinetic

File: urdf/amigo.urdf.xacro (robot description, xacro)
@@ -21,6 +21,6 @@
     <!--========BUILD ARMS======-->
     <xacro:include filename="$(find amigo_description)/urdf/arms/arm.urdf.xacro" />
-    <xacro:arm whichside="right" sidesign="+1.0" rollsign="+"/>
-    <xacro:arm whichside="left"  sidesign="-1.0" rollsign="-"/>
+    <xacro:arm whichside="right" sidesign="1" rollsign="+"/>
+    <xacro:arm whichside="left"  sidesign="-1" rollsign="-"/>
     <!--extra arm visuals-->
     <xacro:include filename="$(find amigo_description)/urdf/arm_extra_visuals/arm_extra.urdf.xacro" />

File: urdf/arms/arm.urdf.xacro (robot description, xacro)
@@ -4,5 +4,5 @@
     <license>BSD</license>
     <review status="unreviewed" notes=""/>
-    <property name="prefix" value="amigo/"/>
+    <xacro:property name="prefix" value="amigo/"/>
     <!--Start of the macro
     @param whichside is "left"  or "right"

File: urdf/head/head.urdf.xacro (robot description, xacro)
@@ -26,5 +26,4 @@
    <origin xyz="0.0 0.0 0.0335" rpy="0 0 0" />
    <inertia ixx="0.0001"  ixy="0"  ixz="0" iyy="0.0001" iyz="0" izz="0.0001" />
-   <color rgba="0.25 0.25 0.25 1.0"/>
 </xacro:my_link>
 <!-- the link that represents the tilting part of the neck, is above neck_pan -->

Commit message: Only declare prefix once

File: urdf/amigo.urdf.xacro (robot description, xacro)
@@ -4,5 +4,6 @@
     <license>BSD</license>
     <review status="unreviewed" notes=""/>
-    <!--get link & joint definitions -->
+    <xacro:property name="prefix" value="amigo/" scope="parent | global"/>
+        <!--get link & joint definitions -->
     <xacro:include filename="$(find amigo_description)/urdf/macro_definitions.xacro" />
     <!--get custom materials -->

File: urdf/arm_extra_visuals/arm_extra.urdf.xacro (robot description, xacro)
@@ -10,5 +10,4 @@
 it has to be reversable and xml cannot multiply - or + but can multiply
  -1 and +1-->
-    <xacro:property name="prefix" value="amigo/"/>
 <xacro:macro name="arm_extra" params="whichside sidesign rollsign">
 <!--the black cylinder sealing the upper arm-->

File: urdf/arms/arm.urdf.xacro (robot description, xacro)
@@ -4,5 +4,4 @@
     <license>BSD</license>
     <review status="unreviewed" notes=""/>
-    <xacro:property name="prefix" value="amigo/"/>
     <!--Start of the macro
     @param whichside is "left"  or "right"

File: urdf/base/base.urdf.xacro (robot description, xacro)
@@ -3,5 +3,4 @@
     <author>Rein Appeldoorn</author>
     <review status="unreviewed" notes=""/>
-    <xacro:property name="prefix" value="amigo/"/>
     <joint name="base_phi_joint" type="continuous">
         <axis xyz="0 0 1"/>

File: urdf/body_extra_visuals/body_extra.urdf.xacro (robot description, xacro)
@@ -4,5 +4,4 @@
    <license>BSD</license>
    <review status="unreviewed" notes=""/>
-    <xacro:property name="prefix" value="amigo/"/>
 <!--base plate at the bottom of the bottomcovers-->
 <xacro:my_link_textured name="base_plate" mass="0.1" texture="aluminium">

File: urdf/head/head.urdf.xacro (robot description, xacro)
@@ -4,5 +4,4 @@
    <license>BSD</license>
    <review status="unreviewed" notes=""/>
-    <xacro:property name="prefix" value="amigo/"/>
 <!--head-->
 <!-- !!!!!!!!!something without a visual not sure what this is!!!!!!!!!!!! -->

File: urdf/kinect/top_kinect.urdf.xacro (robot description, xacro)
@@ -2,5 +2,4 @@
 <robot xmlns:xacro="http://ros.org/wiki/xacro">
   <xacro:property name="M_PI" value="3.14159"/>
-  <xacro:property name="prefix" value="amigo/"/>
   <joint name="top_kinect/base_kinect_joint" type="fixed">
     <origin xyz="0.035 0.0 0.10" rpy="0.0 0.0 0.025" /> <!-- THESE VALUES ARE ROUGH ESTIMATES!! -->

File: urdf/laser/laser.urdf.xacro (robot description, xacro)
@@ -4,5 +4,4 @@
    <license>BSD</license>
    <review status="unreviewed" notes=""/>
-   <xacro:property name="prefix" value="amigo/"/>
 <!--the laser at the base of the robot -->
 <xacro:my_link name="base_laser" mass="0.5" color="Black">

File: urdf/laser/torso_laser.urdf.xacro (robot description, xacro)
@@ -4,5 +4,4 @@
    <license>BSD</license>
    <review status="unreviewed" notes=""/>
-   <xacro:property name="prefix" value="amigo/"/>
 <xacro:my_link name="torso_dummy" mass="0" color="Red">
    <cylinder radius="0.0" length="0.00" />
