Commit message: updated the top kinect frame back to its previous setting
git-svn-id: https://roboticssrv.wtb.tue.nl/svn/ros/code/tue-ros-pkg/trunk/amigo_common/amigo_description@22372 3a3c2cfb-d3b9-409e-9e75-db8fcdbcaac6

File: urdf/xacro/kinect/top_kinect.urdf.xacro (robot description, xacro)
@@ -6,5 +6,5 @@
   <property name="M_PI" value="3.14159"/>
   <joint name="top_kinect/base_kinect_joint" type="fixed">
-    <origin xyz="0.07 0 0.07" rpy="0 0 0" /> <!-- THESE VALUES ARE ROUGH ESTIMATES!! -->
+    <origin xyz="0.07 0.05 0.10" rpy="0 0.01 0.015" /> <!-- THESE VALUES ARE ROUGH ESTIMATES!! -->
     <parent link="head" />
     <child link="top_kinect/openni_camera" />

Commit message: replaced top kinect and updated params
git-svn-id: https://roboticssrv.wtb.tue.nl/svn/ros/code/tue-ros-pkg/trunk/amigo_common/amigo_description@22635 3a3c2cfb-d3b9-409e-9e75-db8fcdbcaac6

File: urdf/xacro/kinect/top_kinect.urdf.xacro (robot description, xacro)
@@ -6,5 +6,5 @@
   <property name="M_PI" value="3.14159"/>
   <joint name="top_kinect/base_kinect_joint" type="fixed">
-    <origin xyz="0.07 0.05 0.10" rpy="0 0.01 0.015" /> <!-- THESE VALUES ARE ROUGH ESTIMATES!! -->
+    <origin xyz="0.07 0.05 0.10" rpy="0.02 0.05 0.015" /> <!-- THESE VALUES ARE ROUGH ESTIMATES!! -->
     <parent link="head" />
     <child link="top_kinect/openni_camera" />
