Commit message: Suppress the legacy interpretation of sloppy xacro tags

File: urdf/xacro/kinect/base_kinect.urdf.xacro (robot description, xacro)
@@ -4,5 +4,5 @@
       xmlns:interface="http://playerstage.sourceforge.net/gazebo/xmlschema/#interface"
       xmlns:xacro="http://ros.org/wiki/xacro">
-  <property name="M_PI" value="3.14159"/>
+  <xacro:property name="M_PI" value="3.14159"/>
   <joint name="base_kinect/base_kinect_joint" type="fixed">
     <origin xyz="0.3 0 0.26" rpy="0 -0.07 0" /> <!-- THESE VALUES STILL HAVE TO BE CALIBRATED!! -->

File: urdf/xacro/kinect/top_kinect.urdf.xacro (robot description, xacro)
@@ -4,5 +4,5 @@
       xmlns:interface="http://playerstage.sourceforge.net/gazebo/xmlschema/#interface"
       xmlns:xacro="http://ros.org/wiki/xacro">
-  <property name="M_PI" value="3.14159"/>
+  <xacro:property name="M_PI" value="3.14159"/>
   <joint name="top_kinect/base_kinect_joint" type="fixed">
     <origin xyz="0.035 0.0 0.10" rpy="0.0 0.0 0.025" /> <!-- THESE VALUES ARE ROUGH ESTIMATES!! -->
