Commit message: Added spring to remove play in tilt dynamixel
git-svn-id: https://roboticssrv.wtb.tue.nl/svn/ros/trunk/amigo_common/amigo_description@22740 3a3c2cfb-d3b9-409e-9e75-db8fcdbcaac6

File: urdf/xacro/head/head.urdf.xacro (robot description, xacro)
@@ -17,5 +17,5 @@
   <child link="head_mount"/>
   <axis xyz="0 0 1"/>
-  <origin xyz="0.097 0.0 0.0" rpy="  0.0 0.0 0.0"/>
+  <origin xyz="0.11 0.0 0.0" rpy="  0.0 0.0 0.0"/>
 </joint>
 <!-- the link that represents the panning part of the neck, is below neck_tilt -->

File: urdf/xacro/kinect/top_kinect.urdf.xacro (robot description, xacro)
@@ -6,5 +6,5 @@
   <property name="M_PI" value="3.14159"/>
   <joint name="top_kinect/base_kinect_joint" type="fixed">
-    <origin xyz="0.07 0.05 0.10" rpy="0.02 0.05 0.015" /> <!-- THESE VALUES ARE ROUGH ESTIMATES!! -->
+    <origin xyz="0.07 0.05 0.10" rpy="0.02 0.01 0.015" /> <!-- THESE VALUES ARE ROUGH ESTIMATES!! -->
     <parent link="head" />
     <child link="top_kinect/openni_camera" />
