Commit message: Fixed typo
git-svn-id: https://roboticssrv.wtb.tue.nl/svn/ros/code/tue-ros-pkg/trunk/amigo_common/amigo_description@18232 3a3c2cfb-d3b9-409e-9e75-db8fcdbcaac6

File: urdf/xacro/body/body.urdf.xacro (robot description, xacro)
@@ -13,5 +13,5 @@
 </xacro:my_link_texturedmesh>
 <!--the spindle-->
-<xacro:my_link_texturedmesh name="torso_slider" mass="0.1" texture="aluminum">
+<xacro:my_link_texturedmesh name="torso_slider" mass="0.1" texture="aluminium">
    <origin xyz="0 0 0" rpy="0 0 0"/>
    <origin xyz="0.05 0 0.0" rpy="0 0 1.5708"/>

File: urdf/xacro/body_extra_visuals/body_extra.urdf.xacro (robot description, xacro)
@@ -5,5 +5,5 @@
    <review status="unreviewed" notes=""/>
 <!--base plate at the bottom of the bottomcovers-->
-<xacro:my_link_textured name="base_plate" mass="0.1" texture="aluminum">
+<xacro:my_link_textured name="base_plate" mass="0.1" texture="aluminium">
    <cylinder radius="0.333" length="0.02" />
    <origin xyz="0.0 0.0 0.0" rpy="0 0 0"/>
@@ -19,5 +19,5 @@
 <!--the extra sliders next to and behind the spindle-->
 <!--right link-->
-<xacro:my_link_texturedmesh name="torso_assist_slider_right" mass="0.01" texture="aluminum">
+<xacro:my_link_texturedmesh name="torso_assist_slider_right" mass="0.01" texture="aluminium">
    <origin xyz="0 0 0" rpy="0 0 0"/>
    <origin xyz="-0.4  0.0 0.0" rpy="0 1.5708 0"/>
@@ -26,5 +26,5 @@
 </xacro:my_link_texturedmesh>
 <!--left link-->
-<xacro:my_link_texturedmesh name="torso_assist_slider_left" mass="0.01" texture="aluminum">
+<xacro:my_link_texturedmesh name="torso_assist_slider_left" mass="0.01" texture="aluminium">
    <origin xyz="0 0 0" rpy="0 0 0"/>
    <origin xyz="-0.4  0.0 0.0" rpy="0 1.5708 0"/>
@@ -33,5 +33,5 @@
 </xacro:my_link_texturedmesh>
 <!--back link-->
-<xacro:my_link_texturedmesh name="torso_assist_slider_back" mass="0.01" texture="aluminum">
+<xacro:my_link_texturedmesh name="torso_assist_slider_back" mass="0.01" texture="aluminium">
    <origin xyz="0 0 0" rpy="0 0 0"/>
    <origin xyz="-0.4 0.0 0.0" rpy="0 1.5708 0"/>

File: urdf/xacro/head/head.urdf.xacro (robot description, xacro)
@@ -28,5 +28,5 @@
 </xacro:my_link>
 <!-- the link that represents the tilting part of the neck, is above neck_pan -->
-<xacro:my_link_texturedmesh name="neck_tilt" mass="0.05" texture="aluminum">
+<xacro:my_link_texturedmesh name="neck_tilt" mass="0.05" texture="aluminium">
    <origin xyz="0.0 -0.0 0.0285" rpy="0 0 0"/>
    <origin xyz="0.0 -0.0 0.015" rpy="0 0 0" />

File: urdf/xacro/materials.urdf.xacro (robot description, xacro)
@@ -38,6 +38,6 @@
     <texture filename="package://amigo_description/media/materials/textures/logo/tue.jpg" />
   </material>
-  <material name="amigo_description/aluminum">
-    <texture filename="package://amigo_description/media/materials/textures/aluminum/aluminium_0001_c.jpg" />
+  <material name="amigo_description/aluminium">
+    <texture filename="package://amigo_description/media/materials/textures/aluminium/aluminium_0001_c.jpg" />
   </material>
   <material name="amigo_description/orange">

Commit message: Fixed torso: effort limit was too low
git-svn-id: https://roboticssrv.wtb.tue.nl/svn/ros/code/tue-ros-pkg/trunk/amigo_common/amigo_description@18252 3a3c2cfb-d3b9-409e-9e75-db8fcdbcaac6

File: urdf/xacro/body/body.urdf.xacro (robot description, xacro)
@@ -40,5 +40,5 @@
   <origin xyz="0.0 0.0 0.58" rpy="3.14159265 -1.5708 0"/>
   <dynamics damping="3" friction="0.0"/> <!--*-->
-  <limit effort="30" velocity="1.0" lower="0.0" upper="0.41" /> <!--*-->
+  <limit effort="1000" velocity="10.0" lower="0.0" upper="0.41" /> <!--*-->
 </joint>
 <joint name="base_link_joint" type="fixed">

Commit message: Fixed URDF error

File: urdf/xacro/body/body.urdf.xacro (robot description, xacro)
@@ -27,10 +27,10 @@
 </xacro:my_link_texturedmesh>
 <!--the root of the tf-tree, because it serves only this function it has no visuals-->
-<xacro:my_link name="base_link" mass="0" color="Red">
+<link name="base_link" type="planar">
    <cylinder radius="0.0" length="0.00" />
    <origin xyz="0.0 0.0 0.0" rpy="0 0 0"/>
    <origin xyz="0.0 0.0 0.0" rpy="0 0 0" />
    <inertia ixx="0"  ixy="0"  ixz="0" iyy="0" iyz="0" izz="0" />
-</xacro:my_link>
+</link>
 <!-- joints start here -->
 <joint name="torso_joint" type="prismatic">
