Commit message: Removed TF prefix

File: urdf/arm_extra_visuals/arm_extra.urdf.xacro (robot description, xacro)
@@ -10,4 +10,5 @@
 it has to be reversable and xml cannot multiply - or + but can multiply
  -1 and +1-->
+    <xacro:property name="prefix" value="amigo/"/>
 <xacro:macro name="arm_extra" params="whichside sidesign rollsign">
 <!--the black cylinder sealing the upper arm-->
@@ -55,31 +56,31 @@
 <!--the joints start here-->
 <joint name="upper_arm_top_joint_${whichside}" type="fixed">
-  <parent link="upper_arm_${whichside}" />
-  <child link="upper_arm_top_${whichside}"/>
+  <parent link="${prefix}upper_arm_${whichside}" />
+  <child link="${prefix}upper_arm_top_${whichside}"/>
   <origin xyz="-0.01 -0.1 0.0" rpy="1.5708 0 0.0"/>
 </joint>
 <joint name="elbow_extra_block_joint_${whichside}" type="fixed">
-  <parent link="upper_arm_${whichside}"/>
-  <child link="elbow_extra_block_${whichside}"/>
+  <parent link="${prefix}upper_arm_${whichside}"/>
+  <child link="${prefix}elbow_extra_block_${whichside}"/>
   <origin xyz="0.0 -0.31 0.0" rpy="-1.5708 0 0"/>
 </joint>
 <joint name="elbow_extra_block2_joint_${whichside}" type="fixed">
-  <parent link="upper_arm_${whichside}"/>
-  <child link="elbow_extra_block2_${whichside}"/>
+  <parent link="${prefix}upper_arm_${whichside}"/>
+  <child link="${prefix}elbow_extra_block2_${whichside}"/>
   <origin xyz="0.0 -0.31 0.0" rpy="-1.5708 0 0"/>
 </joint>
 <joint name="fore_arm_top_joint_${whichside}" type="fixed" >
-  <parent link="fore_arm_${whichside}"/>
-  <child link="fore_arm_top_${whichside}"/>
+  <parent link="${prefix}fore_arm_${whichside}"/>
+  <child link="${prefix}fore_arm_top_${whichside}"/>
    <origin xyz="0.002 -0.011 0.0" rpy="1.5708 0 0"/>
 </joint>
 <joint name="wrist_visual_joint_${whichside}" type="fixed">
-  <parent link="wrist_link6_${whichside}"/>
-  <child link="wrist_visual_${whichside}"/>
+  <parent link="${prefix}wrist_link6_${whichside}"/>
+  <child link="${prefix}wrist_visual_${whichside}"/>
   <origin xyz="-0.02 0.0 0.0" rpy="1.5708 0 0"/>
 </joint>
 <joint name="wrist_to_hand_block_joint_${whichside}" type="fixed">
-  <parent link="wrist_link6_${whichside}"/>
-  <child link="wrist_to_hand_block_${whichside}"/>
+  <parent link="${prefix}wrist_link6_${whichside}"/>
+  <child link="${prefix}wrist_to_hand_block_${whichside}"/>
   <origin xyz="0.0 0.0 0.0" rpy="0 0 0"/>
 </joint>

File: urdf/base/base.urdf.xacro (robot description, xacro)
@@ -3,13 +3,14 @@
     <author>Rein Appeldoorn</author>
     <review status="unreviewed" notes=""/>
+    <xacro:property name="prefix" value="amigo/"/>
     <joint name="base_phi_joint" type="continuous">
         <axis xyz="0 0 1"/>
-        <parent link="base_y_link"/>
+        <parent link="${prefix}base_y_link"/>
         <origin rpy="0 0 0" xyz="0 0 0"/>
-        <child link="base_link"/>
+        <child link="${prefix}base_link"/>
         <dynamics damping="100" friction="20" />
 	<limit effort="1000" velocity="1000" lower="-1000" upper="1000" />
     </joint>
-    <link name="base_y_link">
+    <link name="${prefix}base_y_link">
         <inertial>
             <mass value="10"/>
@@ -20,11 +21,11 @@
     <joint name="base_y_joint" type="prismatic">
         <axis xyz="0 1 0" />
-        <parent link="base_x_link" />
+        <parent link="${prefix}base_x_link" />
         <origin rpy="0 0 0" xyz="0 0 0" />
-        <child link="base_y_link" />
+        <child link="${prefix}base_y_link" />
         <dynamics damping="100" friction="20" />
         <limit effort="1000" velocity="1000" lower="-1000" upper="1000" />
     </joint>
-    <link name="base_x_link">
+    <link name="${prefix}base_x_link">
         <inertial>
             <mass value="10"/>
@@ -35,11 +36,11 @@
     <joint name="base_x_joint" type="prismatic">
         <axis xyz="1 0 0" />
-        <parent link="base_fixed_link" />
+        <parent link="${prefix}base_fixed_link" />
         <origin rpy="0 0 0" xyz="0 0 0" />
-        <child link="base_x_link" />
+        <child link="${prefix}base_x_link" />
         <dynamics damping="100" friction="20" />
 	<limit effort="1000" velocity="1000" lower="-1000" upper="1000" />
     </joint>
-    <link name="base_fixed_link">
+    <link name="${prefix}base_fixed_link">
         <inertial>
             <mass value="10"/>
@@ -51,5 +52,5 @@
         <parent link="world" />
         <origin rpy="0 0 0" xyz="0 0 0" />
-        <child link="base_fixed_link" />
+        <child link="${prefix}base_fixed_link" />
     </joint>
     <link name="world" />

File: urdf/body_extra_visuals/body_extra.urdf.xacro (robot description, xacro)
@@ -4,4 +4,5 @@
    <license>BSD</license>
    <review status="unreviewed" notes=""/>
+    <xacro:property name="prefix" value="amigo/"/>
 <!--base plate at the bottom of the bottomcovers-->
 <xacro:my_link_textured name="base_plate" mass="0.1" texture="aluminium">
@@ -12,6 +13,6 @@
 </xacro:my_link_textured>
   <joint name="base_plate_joint" type="fixed">
-    <parent link="base_link"/>
-    <child link="base_plate"/>
+    <parent link="${prefix}base_link"/>
+    <child link="${prefix}base_plate"/>
     <axis xyz="1 0 0"/>
     <origin xyz="0.0 0.0 0.05" rpy="0 0 0"/>
@@ -41,18 +42,18 @@
 <!--left joint-->
 <joint name="torso_slider_assist_joint_right" type="fixed">
-    <parent link="torso"/>
-    <child link="torso_assist_slider_right"/>
+    <parent link="${prefix}torso"/>
+    <child link="${prefix}torso_assist_slider_right"/>
     <origin xyz="-0.3 0.1 0.0" rpy="0 0 0"/>
 </joint>
 <!--right joint-->
 <joint name="torso_slider_assist_joint_left" type="fixed">
-    <parent link="torso"/>
-    <child link="torso_assist_slider_left"/>
+    <parent link="${prefix}torso"/>
+    <child link="${prefix}torso_assist_slider_left"/>
     <origin xyz="-0.3 -0.1 0.0" rpy="0 0 0"/>
 </joint>
 <!--back joint-->
 <joint name="torso_slider_assist_joint_back" type="fixed">
-    <parent link="torso"/>
-    <child link="torso_assist_slider_back"/>
+    <parent link="${prefix}torso"/>
+    <child link="${prefix}torso_assist_slider_back"/>
     <origin xyz="-0.3 0.0 -0.1" rpy="1.5708 0 0"/>
 </joint>
@@ -65,6 +66,6 @@
 </xacro:my_link>
 <joint name="clavicle_joint" type="fixed">
-    <parent link="torso"/>
-    <child link="clavicles"/>
+    <parent link="${prefix}torso"/>
+    <child link="${prefix}clavicles"/>
     <origin xyz="0.05 0.0 0.0" rpy="0 0 0"/>
 </joint>

File: urdf/head/head.urdf.xacro (robot description, xacro)
@@ -4,7 +4,8 @@
    <license>BSD</license>
    <review status="unreviewed" notes=""/>
+    <xacro:property name="prefix" value="amigo/"/>
 <!--head-->
 <!-- !!!!!!!!!something without a visual not sure what this is!!!!!!!!!!!! -->
-<link name="head_mount">
+<link name="${prefix}head_mount">
   <inertial>
     <origin xyz="0.0 0.0 0.0" rpy="0 0 0"/>
@@ -14,6 +15,6 @@
 </link>
 <joint name="head_mount_joint" type="fixed">
-  <parent link="torso"/>
-  <child link="head_mount"/>
+  <parent link="${prefix}torso"/>
+  <child link="${prefix}head_mount"/>
   <axis xyz="0 0 1"/>
   <origin xyz="0.11 0.0 0.0426" rpy="0.0 0.0 0.0"/>
@@ -42,6 +43,6 @@
   </my_link_texturedmesh>
   <joint name="head_joint" type="fixed">
-    <parent link="neck_tilt"/>
-    <child link="head"/>
+    <parent link="${prefix}neck_tilt"/>
+    <child link="${prefix}head"/>
   </joint>
 <!-- the tilt and pan joints-->

File: urdf/kinect/top_kinect.urdf.xacro (robot description, xacro)
@@ -2,11 +2,12 @@
 <robot xmlns:xacro="http://ros.org/wiki/xacro">
   <xacro:property name="M_PI" value="3.14159"/>
+  <xacro:property name="prefix" value="amigo/"/>
   <joint name="top_kinect/base_kinect_joint" type="fixed">
     <origin xyz="0.035 0.0 0.10" rpy="0.0 0.0 0.025" /> <!-- THESE VALUES ARE ROUGH ESTIMATES!! -->
     <origin xyz="0.035 0.0 0.10" rpy="0.0 0.0 0.025" /> <!-- THESE VALUES ARE ROUGH ESTIMATES!! -->
-    <parent link="head" />
-    <child link="top_kinect/openni_camera" />
+    <parent link="${prefix}head" />
+    <child link="${prefix}top_kinect/openni_camera" />
   </joint>
-  <link name="top_kinect/openni_camera">
+  <link name="${prefix}top_kinect/openni_camera">
     <inertial>
       <mass value="0.01" />
@@ -33,8 +34,8 @@
   <joint name="top_kinect/kinect_depth_joint" type="fixed">
     <origin xyz="0 0.0125 0" rpy="0 0 0" />
-    <parent link="top_kinect/openni_camera" />
-    <child link="top_kinect/openni_depth_frame" />
+    <parent link="${prefix}top_kinect/openni_camera" />
+    <child link="${prefix}top_kinect/openni_depth_frame" />
   </joint>
-  <link name="top_kinect/openni_depth_frame">
+  <link name="${prefix}top_kinect/openni_depth_frame">
     <inertial>
       <mass value="0.01" />
@@ -47,8 +48,8 @@
   <joint name="top_kinect/kinect_depth_optical_joint" type="fixed">
     <origin xyz="0 0 0" rpy="${-M_PI/2} 0 ${-M_PI/2}" />
-    <parent link="top_kinect/openni_depth_frame" />
-    <child link="top_kinect/openni_depth_optical_frame" />
+    <parent link="${prefix}top_kinect/openni_depth_frame" />
+    <child link="${prefix}top_kinect/openni_depth_optical_frame" />
   </joint>
-  <link name="top_kinect/openni_depth_optical_frame">
+  <link name="${prefix}top_kinect/openni_depth_optical_frame">
     <inertial>
       <mass value="0.001" />
@@ -61,8 +62,8 @@
   <joint name="top_kinect/kinect_rgb_joint" type="fixed">
     <origin xyz="0 -0.0125 0" rpy="0 0 0" />
-    <parent link="top_kinect/openni_camera" />
-    <child link="top_kinect/openni_rgb_frame" />
+    <parent link="${prefix}top_kinect/openni_camera" />
+    <child link="${prefix}top_kinect/openni_rgb_frame" />
   </joint>
-  <link name="top_kinect/openni_rgb_frame">
+  <link name="${prefix}top_kinect/openni_rgb_frame">
     <inertial>
       <mass value="0.001" />
@@ -75,8 +76,8 @@
   <joint name="top_kinect/kinect_rgb_optical_joint" type="fixed">
     <origin xyz="0 0 0" rpy="${-M_PI/2} 0 ${-M_PI/2}" />
-    <parent link="top_kinect/openni_rgb_frame" />
-    <child link="top_kinect/openni_rgb_optical_frame" />
+    <parent link="${prefix}top_kinect/openni_rgb_frame" />
+    <child link="${prefix}top_kinect/openni_rgb_optical_frame" />
   </joint>
-  <link name="top_kinect/openni_rgb_optical_frame">
+  <link name="${prefix}top_kinect/openni_rgb_optical_frame">
     <inertial>
       <mass value="0.001" />

File: urdf/laser/laser.urdf.xacro (robot description, xacro)
@@ -4,4 +4,5 @@
    <license>BSD</license>
    <review status="unreviewed" notes=""/>
+   <xacro:property name="prefix" value="amigo/"/>
 <!--the laser at the base of the robot -->
 <xacro:my_link name="base_laser" mass="0.5" color="Black">
@@ -25,6 +26,6 @@
 </xacro:my_link_textured>
 <joint name="lasertop_joint" type="fixed">
-    <parent link="base_laser"/>
-    <child link="lasertop"/>
+    <parent link="${prefix}base_laser"/>
+    <child link="${prefix}lasertop"/>
 </joint>
 <!--the tue logo in front of the laser-->
@@ -36,6 +37,6 @@
 </xacro:my_link_texturedmesh>
   <joint name="logo_joint" type="fixed">
-    <parent link="base_laser"/>
-    <child link="logo"/>
+    <parent link="${prefix}base_laser"/>
+    <child link="${prefix}logo"/>
   </joint>
 </robot>

File: urdf/laser/torso_laser.urdf.xacro (robot description, xacro)
@@ -4,4 +4,5 @@
    <license>BSD</license>
    <review status="unreviewed" notes=""/>
+   <xacro:property name="prefix" value="amigo/"/>
 <xacro:my_link name="torso_dummy" mass="0" color="Red">
    <cylinder radius="0.0" length="0.00" />
@@ -40,6 +41,6 @@
 </xacro:my_link_textured>
 <joint name="torso_lasertop_joint" type="fixed">
-    <parent link="torso_laser"/>
-    <child link="torso_lasertop"/>
+    <parent link="${prefix}torso_laser"/>
+    <child link="${prefix}torso_lasertop"/>
 </joint>
 </robot>

File: urdf/macro_definitions.xacro (robot description, xacro)
@@ -7,5 +7,5 @@
 <!--use this type of link for standard shapes (bos, cylinder, sphere) with standard color -->
 <xacro:macro name="my_link" params="name mass color *type *origin *visualorigin *inertia">
-  <link name="${name}">
+  <link name="amigo/${name}">
    <inertial>
      <xacro:insert_block name="origin" />
@@ -31,5 +31,5 @@
 <!-- use this type of link if you want the standard shapes with a texture -->
 <xacro:macro name="my_link_textured" params="name mass texture *type *origin *visualorigin *inertia">
-  <link name="${name}">
+  <link name="amigo/${name}">
    <inertial>
      <xacro:insert_block name="origin" />
@@ -55,5 +55,5 @@
 <!--use this type of link for shapes that need to be collision free and thereby also invisible -->
 <xacro:macro name="my_link_coll_free" params="name mass color *type *origin *visualorigin *inertia">
-  <link name="${name}">
+  <link name="amigo/${name}">
    <inertial>
      <xacro:insert_block name="origin" />
@@ -73,5 +73,5 @@
 <!--use this type of link if you want to load a mesh with a standard color -->
 <xacro:macro name="my_link_mesh" params="name mass color *origin *visualorigin *inertia *mesh">
-  <link name="${name}">
+  <link name="amigo/${name}">
    <inertial>
      <xacro:insert_block name="origin" />
@@ -97,5 +97,5 @@
 <!-- use this type of link if you want to load a mesh with a texture -->
 <xacro:macro name="my_link_texturedmesh" params="name mass texture *origin *visualorigin *inertia *mesh">
-  <link name="${name}">
+  <link name="amigo/${name}">
    <inertial>
      <xacro:insert_block name="origin" />
@@ -120,5 +120,5 @@
 <!-- use this type of link if you want a mesh with texture and a different bouding box (then the box around the mesh itself) -->
 <xacro:macro name="my_link_texturedmesh_diff_coll" params="name mass texture *origin *visualorigin *collorigin *inertia *mesh *type">
-  <link name="${name}">
+  <link name="amigo/${name}">
    <inertial>
      <xacro:insert_block name="origin" />
@@ -144,6 +144,6 @@
 <xacro:macro name="my_joint" params="name type parent child *origin *dynamics *axis *limit">
  <joint name="${name}" type="${type}">
-    <parent link="${parent}"/>
-    <child link="${child}"/>
+    <parent link="amigo/${parent}"/>
+    <child link="amigo/${child}"/>
     <xacro:insert_block name="origin" />
     <xacro:insert_block name="axis" />
