Commit message: Fixed TF prefixes

File: urdf/arms/arm.urdf.xacro (robot description, xacro)
@@ -4,4 +4,5 @@
     <license>BSD</license>
     <review status="unreviewed" notes=""/>
+    <property name="prefix" value="amigo/"/>
     <!--Start of the macro
     @param whichside is "left"  or "right"
@@ -136,6 +137,6 @@
     <!--the joints start here-->
       <joint name="shoulder_mount_joint_${whichside}" type="fixed">
-        <parent link="torso"/>
-        <child link="shoulder_mount_${whichside}"/>
+        <parent link="${prefix}torso"/>
+        <child link="${prefix}shoulder_mount_${whichside}"/>
         <origin xyz="0.05 ${sidesign*0.22} 0.0" rpy="0 0 0.0"/>
       </joint>
@@ -189,6 +190,6 @@
     </xacro:my_joint>
     <joint name="finger1_phalanx_joint_${whichside}" type="fixed">
-        <parent link="finger1_${whichside}"/>
-        <child link="finger1_phalanx_${whichside}"/>
+        <parent link="${prefix}finger1_${whichside}"/>
+        <child link="${prefix}finger1_phalanx_${whichside}"/>
         <origin xyz="0 0 -0.06" rpy="0 1.57 0"/>
     </joint>
@@ -200,6 +201,6 @@
     </xacro:my_joint>
     <joint name="finger1_tip_phalanx_joint_${whichside}" type="fixed">
-        <parent link="finger1_tip_${whichside}"/>
-        <child link="finger1_tip_phalanx_${whichside}"/>
+        <parent link="${prefix}finger1_tip_${whichside}"/>
+        <child link="${prefix}finger1_tip_phalanx_${whichside}"/>
         <origin xyz="0 0 -0.06" rpy="0 1.57 0"/>
     </joint>
@@ -211,6 +212,6 @@
     </xacro:my_joint>
     <joint name="finger2_phalanx_joint_${whichside}" type="fixed">
-        <parent link="finger2_${whichside}"/>
-        <child link="finger2_phalanx_${whichside}"/>
+        <parent link="${prefix}finger2_${whichside}"/>
+        <child link="${prefix}finger2_phalanx_${whichside}"/>
         <origin xyz="0 0 -0.06" rpy="0 1.57 0"/>
     </joint>
@@ -222,11 +223,11 @@
     </xacro:my_joint>
     <joint name="finger2_tip_phalanx_joint_${whichside}" type="fixed">
-        <parent link="finger2_tip_${whichside}"/>
-        <child link="finger2_tip_phalanx_${whichside}"/>
+        <parent link="${prefix}finger2_tip_${whichside}"/>
+        <child link="${prefix}finger2_tip_phalanx_${whichside}"/>
         <origin xyz="0 0 -0.06" rpy="0 1.57 0"/>
     </joint>
     <joint name="grippoint_joint_${whichside}" type="fixed">
-      <parent link="hand_${whichside}"/>
-      <child link="grippoint_${whichside}"/>
+      <parent link="${prefix}hand_${whichside}"/>
+      <child link="${prefix}grippoint_${whichside}"/>
       <origin xyz="0.14 0.0 0.0" rpy="0 0 0"/>
     </joint>

File: urdf/body/body.urdf.xacro (robot description, xacro)
@@ -27,14 +27,14 @@
     </xacro:my_link_texturedmesh>
     <!--the root of the tf-tree, because it serves only this function it has no visuals-->
-    <xacro:my_link name="base_link" mass="0" color="Red">
+    <link name="${prefix}base_link" mass="0" color="Red">
        <cylinder radius="0.0" length="0.00" />
        <origin xyz="0.0 0.0 0.0" rpy="0 0 0"/>
        <origin xyz="0.0 0.0 0.0" rpy="0 0 0" />
        <inertia ixx="0"  ixy="0"  ixz="0" iyy="0" iyz="0" izz="0" />
-    </xacro:my_link>
+    </link>
     <!-- joints start here -->
     <joint name="torso_joint" type="prismatic">
-      <parent link="base"/>
-      <child link="torso_slider"/>
+      <parent link="${prefix}base"/>
+      <child link="${prefix}torso_slider"/>
       <axis xyz="1 0 0"/>
       <origin xyz="0.0 0.0 0.58" rpy="3.14159265 -1.5708 0"/>
@@ -43,12 +43,12 @@
     </joint>
     <joint name="base_link_joint" type="fixed">
-      <parent link="base_link"/>
-      <child link="base"/>
+      <parent link="${prefix}base_link"/>
+      <child link="${prefix}base"/>
       <axis xyz="1 0 0"/>
       <origin xyz="0.0 0.0 0.055" rpy="0 0 0"/>
     </joint>
     <joint name="torso_slider_joint" type="fixed">
-      <parent link="torso_slider"/>
-      <child link="torso"/>
+      <parent link="${prefix}torso_slider"/>
+      <child link="${prefix}torso"/>
       <axis xyz="1 0 0"/>
       <origin xyz="0.1 0.0 0.0" rpy="0 0 0"/>

Commit message: Temp restriction on wrist movements

File: urdf/arms/arm.urdf.xacro (robot description, xacro)
@@ -175,5 +175,5 @@
        <dynamics damping="0.35" friction="0.63"/>
        <axis xyz="0 -1 0"/>
-       <limit effort="0.5" velocity="1.0" lower="-0.95" upper="0.95"/>
+       <limit effort="0.5" velocity="1.0" lower="-0.1" upper="0.1"/><!--Only for MoveIt temporarily-->
     </xacro:my_joint>
     <xacro:my_joint name="wrist_yaw_joint_${whichside}" type="revolute" parent="wrist_link6_${whichside}" child="hand_${whichside}">
@@ -181,5 +181,5 @@
        <dynamics damping="0.3" friction="0.68"/>
        <axis xyz="0 0 ${sidesign}1"/>
-       <limit effort="0.5" velocity="1.0" lower="-0.61" upper="0.61"/>
+       <limit effort="0.5" velocity="1.0" lower="-0.1" upper="0.1"/><!--Only for MoveIt temporarily-->
     </xacro:my_joint>
     <xacro:my_joint name="finger1_joint_${whichside}" type="revolute" parent="hand_${whichside}" child="finger1_${whichside}">

Commit message: Reverted Tims temporary change ;)

File: urdf/arms/arm.urdf.xacro (robot description, xacro)
@@ -175,5 +175,5 @@
        <dynamics damping="0.35" friction="0.63"/>
        <axis xyz="0 -1 0"/>
-       <limit effort="0.5" velocity="1.0" lower="-0.1" upper="0.1"/><!--Only for MoveIt temporarily-->
+       <limit effort="0.5" velocity="1.0" lower="-0.95" upper="0.95"/>
     </xacro:my_joint>
     <xacro:my_joint name="wrist_yaw_joint_${whichside}" type="revolute" parent="wrist_link6_${whichside}" child="hand_${whichside}">
@@ -181,5 +181,5 @@
        <dynamics damping="0.3" friction="0.68"/>
        <axis xyz="0 0 ${sidesign}1"/>
-       <limit effort="0.5" velocity="1.0" lower="-0.1" upper="0.1"/><!--Only for MoveIt temporarily-->
+       <limit effort="0.5" velocity="1.0" lower="-0.61" upper="0.61"/>
     </xacro:my_joint>
     <xacro:my_joint name="finger1_joint_${whichside}" type="revolute" parent="hand_${whichside}" child="finger1_${whichside}">
