Commit message: Removed deprecated files and statements; also added xacro run cmake commands

File: urdf/kinect/top_kinect.urdf.xacro (robot description, xacro)
@@ -1,7 +1,4 @@
 <?xml version="1.0"?>
-<root xmlns:sensor="http://playerstage.sourceforge.net/gazebo/xmlschema/#sensor"
-      xmlns:controller="http://playerstage.sourceforge.net/gazebo/xmlschema/#controller"
-      xmlns:interface="http://playerstage.sourceforge.net/gazebo/xmlschema/#interface"
-      xmlns:xacro="http://ros.org/wiki/xacro">
+<robot xmlns:xacro="http://ros.org/wiki/xacro">
   <property name="M_PI" value="3.14159"/>
   <joint name="top_kinect/base_kinect_joint" type="fixed">
@@ -90,3 +87,3 @@
     </inertial>
   </link>
-</root>
+</robot>

File: urdf/macro_definitions.xacro (robot description, xacro)
@@ -28,8 +28,4 @@
     </collision>
   </link>
-<gazebo reference="${name}">
-      <material>Gazebo/${color}</material>
-      <turnGravityOff>false</turnGravityOff>
-    </gazebo>
 </xacro:macro>
 <!-- use this type of link if you want the standard shapes with a texture -->
@@ -56,8 +52,4 @@
     </collision>
   </link>
-<gazebo reference="${name}">
-      <material>amigo_description/${texture}</material>
-      <turnGravityOff>false</turnGravityOff>
-    </gazebo>
 </xacro:macro>
 <!--use this type of link for shapes that need to be collision free and thereby also invisible -->
@@ -78,8 +70,4 @@
     </visual>
   </link>
-<gazebo reference="${name}">
-      <material>Gazebo/${color}</material>
-      <turnGravityOff>false</turnGravityOff>
-    </gazebo>
 </xacro:macro>
 <!--use this type of link if you want to load a mesh with a standard color -->
@@ -106,8 +94,4 @@
     </collision>
   </link>
-<gazebo reference="${name}">
-      <material>Gazebo/${color}</material>
-      <turnGravityOff>false</turnGravityOff>
-    </gazebo>
 </xacro:macro>
 <!-- use this type of link if you want to load a mesh with a texture -->
@@ -133,8 +117,4 @@
     </collision>
   </link>
-<gazebo reference="${name}">
-	  <material>amigo_description/${texture}</material>
-      <turnGravityOff>false</turnGravityOff>
-    </gazebo>
 </xacro:macro>
 <!-- use this type of link if you want a mesh with texture and a different bouding box (then the box around the mesh itself) -->
@@ -160,8 +140,4 @@
     </collision>
   </link>
-<gazebo reference="${name}">
-	  <material>amigo_description/${texture}</material>
-      <turnGravityOff>false</turnGravityOff>
-    </gazebo>
 </xacro:macro>
 <!-- *************** JOINT Definition *****************-->

Commit message: Last mm correction

File: urdf/kinect/top_kinect.urdf.xacro (robot description, xacro)
@@ -3,6 +3,6 @@
   <xacro:property name="M_PI" value="3.14159"/>
   <joint name="top_kinect/base_kinect_joint" type="fixed">
-    <origin xyz="0.035 0.0 0.106" rpy="0.0 0.0 0.025" /> <!-- THESE VALUES ARE ROUGH ESTIMATES!! -->
-    <origin xyz="0.035 0.0 0.106" rpy="0.0 0.0 0.025" /> <!-- THESE VALUES ARE ROUGH ESTIMATES!! -->
+    <origin xyz="0.035 0.0 0.107" rpy="0.0 0.0 0.025" /> <!-- THESE VALUES ARE ROUGH ESTIMATES!! -->
+    <origin xyz="0.035 0.0 0.107" rpy="0.0 0.0 0.025" /> <!-- THESE VALUES ARE ROUGH ESTIMATES!! -->
     <parent link="${prefix}head" />
     <child link="${prefix}top_kinect/openni_camera" />
