Commit message: new head

File: urdf/head/head.urdf.xacro (robot description, xacro)
@@ -21,7 +21,7 @@
 <!-- the link that represents the panning part of the neck, is below neck_tilt -->
 <xacro:my_link name="neck_pan" mass="0.05" color="Black">
-   <cylinder radius="0.015" length="0.0525" />
-   <origin xyz="0.0 0.0 0.0335" rpy="0 0 0"/>
-   <origin xyz="0.0 0.0 0.0335" rpy="0 0 0" />
+   <cylinder radius="0.015" length="0.0855" />
+   <origin xyz="0.0 0.0 0.0520" rpy="0 0 0"/>
+   <origin xyz="0.0 0.0 0.0520" rpy="0 0 0" />
    <inertia ixx="0.0001"  ixy="0"  ixz="0" iyy="0.0001" iyz="0" izz="0.0001" />
 </xacro:my_link>
@@ -52,5 +52,5 @@
 </xacro:my_joint>
 <xacro:my_joint name="neck_tilt_joint" type="revolute" parent="neck_pan" child="neck_tilt">
-   <origin xyz="0.0 0.0 0.0445" rpy="0.0 0.015 0.0"/>
+   <origin xyz="0.0 0.0 0.0775" rpy="0.0 0.015 0.0"/>
    <dynamics damping="0.1" friction="0.0"/>
    <axis xyz="0 1 0"/>

File: urdf/kinect/top_kinect.urdf.xacro (robot description, xacro)
@@ -3,6 +3,6 @@
   <xacro:property name="M_PI" value="3.14159"/>
   <joint name="top_kinect/base_kinect_joint" type="fixed">
-    <origin xyz="0.035 0.0 0.10" rpy="0.0 0.0 0.025" /> <!-- THESE VALUES ARE ROUGH ESTIMATES!! -->
-    <origin xyz="0.035 0.0 0.10" rpy="0.0 0.0 0.025" /> <!-- THESE VALUES ARE ROUGH ESTIMATES!! -->
+    <origin xyz="0.035 0.0 0.106" rpy="0.0 0.0 0.025" /> <!-- THESE VALUES ARE ROUGH ESTIMATES!! -->
+    <origin xyz="0.035 0.0 0.106" rpy="0.0 0.0 0.025" /> <!-- THESE VALUES ARE ROUGH ESTIMATES!! -->
     <parent link="${prefix}head" />
     <child link="${prefix}top_kinect/openni_camera" />

Commit message: head correction

File: urdf/head/head.urdf.xacro (robot description, xacro)
@@ -52,5 +52,5 @@
 </xacro:my_joint>
 <xacro:my_joint name="neck_tilt_joint" type="revolute" parent="neck_pan" child="neck_tilt">
-   <origin xyz="0.0 0.0 0.0775" rpy="0.0 0.015 0.0"/>
+   <origin xyz="0.0 0.0 0.0915" rpy="0.0 0.015 0.0"/>
    <dynamics damping="0.1" friction="0.0"/>
    <axis xyz="0 1 0"/>

Commit message: commit for matthijs, fix of head mount

File: urdf/head/head.urdf.xacro (robot description, xacro)
@@ -17,5 +17,5 @@
   <child link="${prefix}head_mount"/>
   <axis xyz="0 0 1"/>
-  <origin xyz="0.11 0.0 0.0426" rpy="0.0 0.0 0.0"/>
+  <origin xyz="0.11 0.0 0.0426" rpy="0.07 0.0 0.0"/>
 </joint>
 <!-- the link that represents the panning part of the neck, is below neck_tilt -->

Commit message: small fix of head calibration

File: urdf/head/head.urdf.xacro (robot description, xacro)
@@ -17,5 +17,5 @@
   <child link="${prefix}head_mount"/>
   <axis xyz="0 0 1"/>
-  <origin xyz="0.11 0.0 0.0426" rpy="0.07 0.0 0.0"/>
+  <origin xyz="0.11 0.0 0.0426" rpy="0.04 0.0 0.0"/>
 </joint>
 <!-- the link that represents the panning part of the neck, is below neck_tilt -->
