Commit message: Lowered torso acceleration

File: urdf/body/body.urdf.xacro (robot description, xacro)
@@ -40,5 +40,5 @@
       <origin xyz="0.0 0.0 0.58" rpy="3.14159265 -1.5708 0"/>
       <dynamics damping="3" friction="0.0"/> <!--*-->
-      <limit effort="0.1" velocity="0.07" lower="0.09" upper="0.4" />
+      <limit effort="0.07" velocity="0.07" lower="0.09" upper="0.4" />
     </joint>
     <joint name="base_link_joint" type="fixed">

Commit message: feature(manipulation root) added manipulation root frame

File: urdf/body/body.urdf.xacro (robot description, xacro)
@@ -33,4 +33,7 @@
        <inertia ixx="0"  ixy="0"  ixz="0" iyy="0" iyz="0" izz="0" />
     </link>
+    <!-- Root of the kinematic chain. This is used to include additional base DoFs
+    in the manipulation planning -->
+    <link name="${prefix}manipulation_root"/>
     <!-- joints start here -->
     <joint name="torso_joint" type="prismatic">
@@ -48,4 +51,9 @@
       <origin xyz="0.0 0.0 0.055" rpy="0 0 0"/>
     </joint>
+    <joint name="manipulation_joint" type="fixed">
+        <parent link="${prefix}manipulation_root"/>
+        <child link="${prefix}base_link"/>
+        <origin xyz="0 0 0" rpy="0 0 0"/>
+    </joint>
     <joint name="torso_slider_joint" type="fixed">
       <parent link="${prefix}torso_slider"/>

Commit message: Made manipulation joint continous

File: urdf/body/body.urdf.xacro (robot description, xacro)
@@ -51,8 +51,11 @@
       <origin xyz="0.0 0.0 0.055" rpy="0 0 0"/>
     </joint>
-    <joint name="manipulation_joint" type="fixed">
+    <joint name="manipulation_joint" type="continuous">
         <parent link="${prefix}manipulation_root"/>
         <child link="${prefix}base_link"/>
         <origin xyz="0 0 0" rpy="0 0 0"/>
+        <axis xyz="0 0 1"/>
+        <dynamics damping="0.5" friction="1.0"/><!-- ToDo: update?-->
+        <limit effort="3" velocity="1.0"/><!-- ToDo: update!!! -->
     </joint>
     <joint name="torso_slider_joint" type="fixed">

Commit message: chore(urdf): Added matrix

File: urdf/body/body.urdf.xacro (robot description, xacro)
@@ -54,3 +54,13 @@
       <origin xyz="0.1 0.0 0.0" rpy="0 0 0"/>
     </joint>
+    <!-- Matrix creator -->
+    <link name="${prefix}matrix">
+       <origin xyz="0.0 0.0 0.0" rpy="0 0 0" />
+       <inertia ixx="0"  ixy="0"  ixz="0" iyy="0" iyz="0" izz="0" />
+    </link>
+    <joint name="torso_matrix_joint" type="fixed">
+        <parent link="${prefix}torso"/>
+        <child link="${prefix}matrix"/>
+        <origin xyz="0.14 0.0 -0.065" rpy="0 1.5708 0"/>
+    </joint>
 </robot>
